File: HBALLCTRL.kicad_sch (KiCad schematic)
At the start: 9 parts

Commit message: R20260915
Other:
- company: (none) -> Atari
- title: (none) -> PONG
- moved on the sheet: UC1D, UD1A, UE1C, UE1D, UF1, UG1C, UG1D, UH1A, UH1B, UH1C, UH1D, UH2A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

Commit message: R20260918
Parts:
- added R27: R, symbol Device:R_US
- UC1, UD1, UE1, UF1, UG1, UH1, UH2, UH3, UH4: footprint Package_DIP:DIP-14_W7.62mm_Socket_LongPads -> pong:pong_DIP-14_W7.62mm_Socket_LongPads
Connections:
- net +5V: now also R27.1; no longer UH2.8 (J)
- net GND: now also UD1.7 (GND), UF1.10 (GND)
- net VRESET: now also UH1.10
- net +3.3V: now reaches UF1.5 (VCC)
- net +3.3V: now also UD1.14 (VCC)
- net at UH2.12 (C), UH2.9 (C): now also UG1.10
- new net: R27.2, UH2.8 (J)
- no-connect marks 0 -> 2
Other:
- moved on the sheet: UE1D, UG1C, UH2A, UH4A

Commit message: R20260922
Parts:
- R27: footprint (none) -> Resistor_THT:R_Axial_DIN0207_L6.3mm_D2.5mm_P10.16mm_Horizontal
Changed lines of the file:
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@@
 			)
 		)
-		(property "Footprint" ""
+		(property "Footprint" "Resistor_THT:R_Axial_DIN0207_L6.3mm_D2.5mm_P10.16mm_Horizontal"
 			(at 176.276 56.134 90)
 			(hide yes)
