File: HSYNC.kicad_sch (KiCad schematic)
At the start: 12 parts, among them Y1 14.318Mhz

Commit message: R20260915
Parts:
- added R14, R15: R, symbol Device:R_US
- R1, R2: value 330 -> R_US; symbol Device:R -> Device:R_US
Connections:
- net at UF6.11 (K), UF6.8 (J): now also R15.2
- net 128H: now reaches UF6.9 (C), UF7.11, UF9.11 (Q3)
- net 16H: now reaches UF9.1 (~{CKB}), UF9.12 (Q0)
- net GND: now reaches UF9.10 (GND)
- net GND: now also UC9.7 (GND), UC9.7 (GND), UF7.7 (GND), UF8.10 (GND)
- net 8H: now reaches UF8.11 (Q3), UF9.14 (~{CKA})
- net +3.3V: now reaches UF9.5 (VCC)
- net +3.3V: now also UC9.14 (VCC), UC9.14 (VCC), UF7.14 (VCC), UF8.5 (VCC)
- net 64H: now reaches UF7.12, UF9.8 (Q2)
- net 32H: now reaches UF9.9 (Q1)
- net at UF6.1 (J), UF6.13 (~{R}), UF6.4 (K): now also R14.2
- net 4H: now reaches UF7.5, UF8.8 (Q2)
- net 2H: now reaches UF7.6, UF8.9 (Q1)
- net 1H: now reaches UF8.1 (~{CKB}), UF8.12 (Q0)
- new net +5V: R14.1, R15.1
- no-connect marks 0 -> 4
Other:
- company: (none) -> Atari
- title: (none) -> PONG
- moved on the sheet: UE7B, UF6A

Commit message: R20260918
Parts:
- R1, R2: value R_US -> 330
- UC9, UE6, UE7, UF6, UF7, UF8, UF9: footprint Package_DIP:DIP-14_W7.62mm_Socket_LongPads -> pong:pong_DIP-14_W7.62mm_Socket_LongPads
Changed lines of the file:
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@@
-	(wire
-		(pts
-			(xy 120.65 177.8) (xy 129.54 177.8)
-		)
-		(stroke
-			(width 0)
-			(type default)
-		)
-	)
 	(wire
 		(pts
@@
 	(global_label "CLK"
 		(shape input)
-		(at 129.54 177.8 0)
+		(at 120.65 177.8 0)
 		(fields_autoplaced yes)
 		(effects
@@
 		)
 		(property "Intersheetrefs" "${INTERSHEET_REFS}"
-			(at 136.0933 177.8 0)
+			(at 127.2033 177.8 0)
 			(hide yes)
 			(show_name no)
@@
 			)
 		)
-		(property "Footprint" "Package_DIP:DIP-14_W7.62mm_Socket_LongPads"
+		(property "Footprint" "pong:pong_DIP-14_W7.62mm_Socket_LongPads"
 			(at 218.44 58.42 0)
 			(hide yes)
@@
 		)
 		(property "Value" "+3.3V"
-			(at 88.9 146.304 0)
+			(at 93.98 149.86 0)
 			(show_name no)
 			(do_not_autoplace no)
@@
 			)
 		)
-		(property "Value" "R_US"
+		(property "Value" "330"
 			(at 26.67 142.24 90)
 			(show_name no)
@@
 			)
 		)
-		(property "Footprint" "Package_DIP:DIP-14_W7.62mm_Socket_LongPads"
+		(property "Footprint" "pong:pong_DIP-14_W7.62mm_Socket_LongPads"
 			(at 167.64 59.69 0)
 			(hide yes)
@@
 		)
 		(property "Value" "+3.3V"
-			(at 35.56 146.304 0)
+			(at 40.386 148.59 0)
 			(show_name no)
 			(do_not_autoplace no)
@@
 			)
 		)
-		(property "Footprint" "Package_DIP:DIP-14_W7.62mm_Socket_LongPads"
+		(property "Footprint" "pong:pong_DIP-14_W7.62mm_Socket_LongPads"
 			(at 113.03 180.34 0)
 			(hide yes)
@@
 			)
 		)
-		(property "Value" "R_US"
+		(property "Value" "330"
 			(at 99.06 142.24 90)
 			(show_name no)
@@
 			)
 		)
-		(property "Footprint" "Package_DIP:DIP-14_W7.62mm_Socket_LongPads"
+		(property "Footprint" "pong:pong_DIP-14_W7.62mm_Socket_LongPads"
 			(at 63.5 180.34 0)
 			(hide yes)
@@
 			)
 		)
-		(property "Footprint" "Package_DIP:DIP-14_W7.62mm_Socket_LongPads"
+		(property "Footprint" "pong:pong_DIP-14_W7.62mm_Socket_LongPads"
 			(at 35.56 160.02 0)
 			(hide yes)
@@
 			)
 		)
-		(property "Footprint" "Package_DIP:DIP-14_W7.62mm_Socket_LongPads"
+		(property "Footprint" "pong:pong_DIP-14_W7.62mm_Socket_LongPads"
 			(at 88.9 160.02 0)
 			(hide yes)
@@
 			)
 		)
-		(property "Footprint" "Package_DIP:DIP-14_W7.62mm_Socket_LongPads"
+		(property "Footprint" "pong:pong_DIP-14_W7.62mm_Socket_LongPads"
 			(at 196.85 148.59 0)
 			(hide yes)
@@
 			)
 		)
-		(property "Footprint" "Package_DIP:DIP-14_W7.62mm_Socket_LongPads"
+		(property "Footprint" "pong:pong_DIP-14_W7.62mm_Socket_LongPads"
 			(at 161.29 128.27 0)
 			(hide yes)
@@
 			)
 		)
-		(property "Footprint" "Package_DIP:DIP-14_W7.62mm_Socket_LongPads"
+		(property "Footprint" "pong:pong_DIP-14_W7.62mm_Socket_LongPads"
 			(at 105.41 58.42 0)
 			(hide yes)

Commit message: R20260921
Connections:
- net H RESET renamed HRESET
Changed lines of the file:
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@@
-		)
-	)
-	(label "H RESET"
-		(at 207.01 38.1 180)
-		(effects
-			(font
-				(size 1.27 1.27)
-			)
-			(justify right bottom)
 		)
 	)
@@
 			(hide yes)
 			(show_name no)
+			(do_not_autoplace no)
+			(effects
+				(font
+					(size 1.27 1.27)
+				)
+				(justify left)
+			)
+		)
+	)
+	(global_label "HRESET"
+		(shape input)
+		(at 194.31 38.1 90)
+		(fields_autoplaced yes)
+		(effects
+			(font
+				(size 1.27 1.27)
+			)
+			(justify left)
+		)
+		(property "Intersheetrefs" "${INTERSHEET_REFS}"
+			(at 194.31 28.0392 90)
+			(hide yes)
+			(show_name no)

Commit message: R20260922
Parts:
- C1, C2: footprint (none) -> Capacitor_THT:C_Disc_D10.5mm_W5.0mm_P7.50mm
- R1, R14, R15, R2: footprint (none) -> Resistor_THT:R_Axial_DIN0207_L6.3mm_D2.5mm_P10.16mm_Horizontal
- Y1: footprint (none) -> Crystal:Crystal_HC49-U_Vertical
Changed lines of the file:
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@@
 			)
 		)
-		(property "Footprint" ""
+		(property "Footprint" "Capacitor_THT:C_Disc_D10.5mm_W5.0mm_P7.50mm"
 			(at 57.15 160.9852 0)
 			(hide yes)
@@
 			)
 		)
-		(property "Footprint" ""
+		(property "Footprint" "Resistor_THT:R_Axial_DIN0207_L6.3mm_D2.5mm_P10.16mm_Horizontal"
 			(at 26.416 147.066 90)
 			(hide yes)
@@
 			)
 		)
-		(property "Footprint" ""
+		(property "Footprint" "Capacitor_THT:C_Disc_D10.5mm_W5.0mm_P7.50mm"
 			(at 77.47 141.9352 0)
 			(hide yes)
@@
 			)
 		)
-		(property "Footprint" ""
+		(property "Footprint" "Crystal:Crystal_HC49-U_Vertical"
 			(at 36.83 140.97 0)
 			(hide yes)
@@
 			)
 		)
-		(property "Footprint" ""
+		(property "Footprint" "Resistor_THT:R_Axial_DIN0207_L6.3mm_D2.5mm_P10.16mm_Horizontal"
 			(at 206.756 49.784 90)
 			(hide yes)
@@
 			)
 		)
-		(property "Footprint" ""
+		(property "Footprint" "Resistor_THT:R_Axial_DIN0207_L6.3mm_D2.5mm_P10.16mm_Horizontal"
 			(at 98.806 147.066 90)
 			(hide yes)
@@
 			)
 		)
-		(property "Footprint" ""
+		(property "Footprint" "Resistor_THT:R_Axial_DIN0207_L6.3mm_D2.5mm_P10.16mm_Horizontal"
 			(at 101.346 171.704 90)
 			(hide yes)
