File: NET.kicad_sch (KiCad schematic)
At the start: 3 parts

Commit message: R20260915
Parts:
- added R18: R, symbol Device:R_US
Connections:
- net +5V: now also R18.2; no longer UF3.10 (~{R})
- net +3.3V: now reaches UG2.14 (VCC)
- net GND: now reaches UG2.7 (GND)
- new net: R18.1, UF3.10 (~{R})
- no-connect marks 0 -> 1
Other:
- company: (none) -> Atari
- title: (none) -> PONG

Commit message: R20260918
Parts:
- UF3, UG2, UG3: footprint Package_DIP:DIP-14_W7.62mm_Socket_LongPads -> pong:pong_DIP-14_W7.62mm_Socket_LongPads
Changed lines of the file:
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@@
 			)
 		)
-		(property "Footprint" "Package_DIP:DIP-14_W7.62mm_Socket_LongPads"
+		(property "Footprint" "pong:pong_DIP-14_W7.62mm_Socket_LongPads"
 			(at 123.19 104.14 0)
 			(hide yes)
@@
 			)
 		)
-		(property "Footprint" "Package_DIP:DIP-14_W7.62mm_Socket_LongPads"
+		(property "Footprint" "pong:pong_DIP-14_W7.62mm_Socket_LongPads"
 			(at 93.98 104.14 0)
 			(hide yes)
@@
 			)
 		)
-		(property "Footprint" "Package_DIP:DIP-14_W7.62mm_Socket_LongPads"
+		(property "Footprint" "pong:pong_DIP-14_W7.62mm_Socket_LongPads"
 			(at 160.02 96.52 0)
 			(hide yes)

Commit message: R20260922
Parts:
- R18: footprint (none) -> Resistor_THT:R_Axial_DIN0207_L6.3mm_D2.5mm_P10.16mm_Horizontal
Changed lines of the file:
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@@
 			)
 		)
-		(property "Footprint" ""
+		(property "Footprint" "Resistor_THT:R_Axial_DIN0207_L6.3mm_D2.5mm_P10.16mm_Horizontal"
 			(at 94.996 115.824 90)
 			(hide yes)
