File: SCORE1.kicad_sch (KiCad schematic)
At the start: 8 parts

Commit message: Added remainder of sheets
Parts:
- UC5, UC6, UD6: footprint Package_DIP:DIP-16_W10.16mm -> Package_DIP:DIP-16_W7.62mm_Socket_LongPads
- UD2, UE2, UE3, UF2, UG1: footprint Package_DIP:DIP-14_W10.16mm -> Package_DIP:DIP-14_W7.62mm_Socket_LongPads
Changed lines of the file:
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@@
 			)
 		)
-		(property "Footprint" "Package_DIP:DIP-14_W10.16mm"
+		(property "Footprint" "Package_DIP:DIP-14_W7.62mm_Socket_LongPads"
 			(at 168.91 55.88 0)
 			(hide yes)
@@
 			)
 		)
-		(property "Footprint" "Package_DIP:DIP-16_W10.16mm"
+		(property "Footprint" "Package_DIP:DIP-16_W7.62mm_Socket_LongPads"
 			(at 52.07 154.94 0)
 			(hide yes)
@@
 			)
 		)
-		(property "Footprint" "Package_DIP:DIP-16_W10.16mm"
+		(property "Footprint" "Package_DIP:DIP-16_W7.62mm_Socket_LongPads"
 			(at 240.03 147.32 0)
 			(hide yes)
@@
 			)
 		)
-		(property "Footprint" "Package_DIP:DIP-14_W10.16mm"
+		(property "Footprint" "Package_DIP:DIP-14_W7.62mm_Socket_LongPads"
 			(at 142.24 90.17 0)
 			(hide yes)
@@
 			)
 		)
-		(property "Footprint" "Package_DIP:DIP-14_W10.16mm"
+		(property "Footprint" "Package_DIP:DIP-14_W7.62mm_Socket_LongPads"
 			(at 205.74 36.83 0)
 			(hide yes)
@@
 			)
 		)
-		(property "Footprint" "Package_DIP:DIP-14_W10.16mm"
+		(property "Footprint" "Package_DIP:DIP-14_W7.62mm_Socket_LongPads"
 			(at 106.68 53.34 0)
 			(hide yes)
@@
 			)
 		)
-		(property "Footprint" "Package_DIP:DIP-14_W10.16mm"
+		(property "Footprint" "Package_DIP:DIP-14_W7.62mm_Socket_LongPads"
 			(at 106.68 90.17 0)
 			(hide yes)
@@
 			)
 		)
-		(property "Footprint" "Package_DIP:DIP-14_W10.16mm"
+		(property "Footprint" "Package_DIP:DIP-14_W7.62mm_Socket_LongPads"
 			(at 160.02 22.86 0)
 			(hide yes)
@@
 			)
 		)
-		(property "Footprint" "Package_DIP:DIP-14_W10.16mm"
+		(property "Footprint" "Package_DIP:DIP-14_W7.62mm_Socket_LongPads"
 			(at 53.34 54.61 0)
 			(hide yes)
@@
 			)
 		)
-		(property "Footprint" "Package_DIP:DIP-16_W10.16mm"
+		(property "Footprint" "Package_DIP:DIP-16_W7.62mm_Socket_LongPads"
 			(at 144.78 153.67 0)
 			(hide yes)

Commit message: R20260915
Parts:
- added R22, R23: R, symbol Device:R_US
Connections:
- net GND: now also UC5.8 (GND), UC6.8 (GND), UD6.8 (GND), UE2.7 (GND), UE3.7 (GND), UE3.7 (GND), UE3.7 (GND), UF2.7 (GND)
- net +3.3V: now reaches UD6.16 (VCC)
- net +3.3V: now also UC5.16 (VCC), UC6.16 (VCC), UE2.14 (VCC), UE3.14 (VCC), UE3.14 (VCC), UE3.14 (VCC), UF2.14 (VCC)
- net at UC5.3 (~{LT}), UC5.5 (~{RBI}): now also R22.2
- net at UC6.4 (I2a), UC6.6 (I0a): now also R23.2
- new net +5V: R22.1, R23.1
- no-connect marks 0 -> 1
Other:
- company: (none) -> Atari
- title: (none) -> PONG
- moved on the sheet: UF2A, UG1A

Commit message: R20260918
Parts:
- UC5, UC6, UD6: footprint Package_DIP:DIP-16_W7.62mm_Socket_LongPads -> pong:pong_DIP-16_W7.62mm_Socket_LongPads
- UD2, UE2, UE3, UF2, UG1: footprint Package_DIP:DIP-14_W7.62mm_Socket_LongPads -> pong:pong_DIP-14_W7.62mm_Socket_LongPads
Other:
- note added: "PIN 2 MAY BE CONNECTED"
Changed lines of the file:
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@@
 		(company "Atari")
 	)
+	(text "PIN 2 MAY BE CONNECTED"
+		(exclude_from_sim no)
+		(at 26.924 50.038 0)
+		(effects
+			(font
+				(size 1.27 1.27)
+			)
+		)
+	)
 	(junction
 		(at 88.9 63.5)
@@
 			)
 		)
-		(property "Footprint" "Package_DIP:DIP-14_W7.62mm_Socket_LongPads"
+		(property "Footprint" "pong:pong_DIP-14_W7.62mm_Socket_LongPads"
 			(at 168.91 55.88 0)
 			(hide yes)
@@
 			)
 		)
-		(property "Footprint" "Package_DIP:DIP-16_W7.62mm_Socket_LongPads"
+		(property "Footprint" "pong:pong_DIP-16_W7.62mm_Socket_LongPads"
 			(at 52.07 154.94 0)
 			(hide yes)
@@
 			)
 		)
-		(property "Footprint" "Package_DIP:DIP-16_W7.62mm_Socket_LongPads"
+		(property "Footprint" "pong:pong_DIP-16_W7.62mm_Socket_LongPads"
 			(at 240.03 147.32 0)
 			(hide yes)
@@
 			)
 		)
-		(property "Footprint" "Package_DIP:DIP-14_W7.62mm_Socket_LongPads"
+		(property "Footprint" "pong:pong_DIP-14_W7.62mm_Socket_LongPads"
 			(at 142.24 90.17 0)
 			(hide yes)
@@
 			)
 		)
-		(property "Footprint" "Package_DIP:DIP-14_W7.62mm_Socket_LongPads"
+		(property "Footprint" "pong:pong_DIP-14_W7.62mm_Socket_LongPads"
 			(at 195.58 36.83 0)
 			(hide yes)
@@
 			)
 		)
-		(property "Footprint" "Package_DIP:DIP-14_W7.62mm_Socket_LongPads"
+		(property "Footprint" "pong:pong_DIP-14_W7.62mm_Socket_LongPads"
 			(at 106.68 53.34 0)
 			(hide yes)
@@
 			)
 		)
-		(property "Footprint" "Package_DIP:DIP-14_W7.62mm_Socket_LongPads"
+		(property "Footprint" "pong:pong_DIP-14_W7.62mm_Socket_LongPads"
 			(at 106.68 90.17 0)
 			(hide yes)
@@
 			)
 		)
-		(property "Footprint" "Package_DIP:DIP-14_W7.62mm_Socket_LongPads"
+		(property "Footprint" "pong:pong_DIP-14_W7.62mm_Socket_LongPads"
 			(at 170.18 34.29 0)
 			(hide yes)
@@
 			)
 		)
-		(property "Footprint" "Package_DIP:DIP-14_W7.62mm_Socket_LongPads"
+		(property "Footprint" "pong:pong_DIP-14_W7.62mm_Socket_LongPads"
 			(at 53.34 54.61 0)
 			(hide yes)
@@
 			)
 		)
-		(property "Footprint" "Package_DIP:DIP-16_W7.62mm_Socket_LongPads"
+		(property "Footprint" "pong:pong_DIP-16_W7.62mm_Socket_LongPads"
 			(at 144.78 153.67 0)
 			(hide yes)

Commit message: R20260922
Parts:
- R22, R23: footprint (none) -> Resistor_THT:R_Axial_DIN0207_L6.3mm_D2.5mm_P10.16mm_Horizontal
Changed lines of the file:
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@@
 			)
 		)
-		(property "Footprint" ""
+		(property "Footprint" "Resistor_THT:R_Axial_DIN0207_L6.3mm_D2.5mm_P10.16mm_Horizontal"
 			(at 158.496 117.094 90)
 			(hide yes)
@@
 			)
 		)
-		(property "Footprint" ""
+		(property "Footprint" "Resistor_THT:R_Axial_DIN0207_L6.3mm_D2.5mm_P10.16mm_Horizontal"
 			(at 214.376 128.524 90)
 			(hide yes)
