File: SCORE2.kicad_sch (KiCad schematic)
At the start: 9 parts

Commit message: Added remainder of sheets
Parts:
- UC3, UC4, UD2, UD3, UD4, UD5, UE2, UE4, UE5: footprint Package_DIP:DIP-14_W10.16mm -> Package_DIP:DIP-14_W7.62mm_Socket_LongPads
Changed lines of the file:
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@@
 			)
 		)
-		(property "Footprint" "Package_DIP:DIP-14_W10.16mm"
+		(property "Footprint" "Package_DIP:DIP-14_W7.62mm_Socket_LongPads"
 			(at 40.64 88.9 0)
 			(hide yes)
@@
 			)
 		)
-		(property "Footprint" "Package_DIP:DIP-14_W10.16mm"
+		(property "Footprint" "Package_DIP:DIP-14_W7.62mm_Socket_LongPads"
 			(at 86.36 30.48 0)
 			(hide yes)
@@
 			)
 		)
-		(property "Footprint" "Package_DIP:DIP-14_W10.16mm"
+		(property "Footprint" "Package_DIP:DIP-14_W7.62mm_Socket_LongPads"
 			(at 73.66 118.11 0)
 			(hide yes)
@@
 			)
 		)
-		(property "Footprint" "Package_DIP:DIP-14_W10.16mm"
+		(property "Footprint" "Package_DIP:DIP-14_W7.62mm_Socket_LongPads"
 			(at 140.97 143.51 0)
 			(hide yes)
@@
 			)
 		)
-		(property "Footprint" "Package_DIP:DIP-14_W10.16mm"
+		(property "Footprint" "Package_DIP:DIP-14_W7.62mm_Socket_LongPads"
 			(at 72.39 53.34 0)
 			(hide yes)
@@
 			)
 		)
-		(property "Footprint" "Package_DIP:DIP-14_W10.16mm"
+		(property "Footprint" "Package_DIP:DIP-14_W7.62mm_Socket_LongPads"
 			(at 82.55 81.28 0)
 			(hide yes)
@@
 			)
 		)
-		(property "Footprint" "Package_DIP:DIP-14_W10.16mm"
+		(property "Footprint" "Package_DIP:DIP-14_W7.62mm_Socket_LongPads"
 			(at 85.09 168.91 0)
 			(hide yes)
@@
 			)
 		)
-		(property "Footprint" "Package_DIP:DIP-14_W10.16mm"
+		(property "Footprint" "Package_DIP:DIP-14_W7.62mm_Socket_LongPads"
 			(at 142.24 166.37 0)
 			(hide yes)
@@
 			)
 		)
-		(property "Footprint" "Package_DIP:DIP-14_W10.16mm"
+		(property "Footprint" "Package_DIP:DIP-14_W7.62mm_Socket_LongPads"
 			(at 149.86 185.42 0)
 			(hide yes)
@@
 			)
 		)
-		(property "Footprint" "Package_DIP:DIP-14_W10.16mm"
+		(property "Footprint" "Package_DIP:DIP-14_W7.62mm_Socket_LongPads"
 			(at 140.97 90.17 0)
 			(hide yes)
@@
 			)
 		)
-		(property "Footprint" "Package_DIP:DIP-14_W10.16mm"
+		(property "Footprint" "Package_DIP:DIP-14_W7.62mm_Socket_LongPads"
 			(at 142.24 27.94 0)
 			(hide yes)
@@
 			)
 		)
-		(property "Footprint" "Package_DIP:DIP-14_W10.16mm"
+		(property "Footprint" "Package_DIP:DIP-14_W7.62mm_Socket_LongPads"
 			(at 199.39 105.41 0)
 			(hide yes)
@@
 			)
 		)
-		(property "Footprint" "Package_DIP:DIP-14_W10.16mm"
+		(property "Footprint" "Package_DIP:DIP-14_W7.62mm_Socket_LongPads"
 			(at 40.64 118.11 0)
 			(hide yes)
@@
 			)
 		)
-		(property "Footprint" "Package_DIP:DIP-14_W10.16mm"
+		(property "Footprint" "Package_DIP:DIP-14_W7.62mm_Socket_LongPads"
 			(at 140.97 120.65 0)
 			(hide yes)
@@
 			)
 		)
-		(property "Footprint" "Package_DIP:DIP-14_W10.16mm"
+		(property "Footprint" "Package_DIP:DIP-14_W7.62mm_Socket_LongPads"
 			(at 142.24 55.88 0)
 			(hide yes)
@@
 			)
 		)
-		(property "Footprint" "Package_DIP:DIP-14_W10.16mm"
+		(property "Footprint" "Package_DIP:DIP-14_W7.62mm_Socket_LongPads"
 			(at 39.37 67.31 0)
 			(hide yes)

Commit message: R20260915
Parts:
- added R24: R, symbol Device:R_US
Connections:
- net +3.3V: now reaches UE4.14 (VCC)
- net +3.3V: now also UC4.14 (VCC), UD3.14 (VCC), UD4.14 (VCC), UD4.14 (VCC), UD4.14 (VCC), UD5.14 (VCC), UD5.14 (VCC), UD5.14 (VCC), UE2.14 (VCC), UE4.14 (VCC), UE4.14 (VCC), UE5.14 (VCC), UE5.14 (VCC)
- net GND: now reaches UE4.7 (GND)
- net GND: now also UC4.7 (GND), UD3.7 (GND), UD4.7 (GND), UD4.7 (GND), UD4.7 (GND), UD5.7 (GND), UD5.7 (GND), UD5.7 (GND), UE2.7 (GND), UE4.7 (GND), UE4.7 (GND), UE5.7 (GND), UE5.7 (GND)
- net at UD3.1: now also R24.2
- new net +5V: R24.1
Other:
- company: (none) -> Atari
- title: (none) -> PONG
- moved on the sheet: UC3D, UC4C, UD3, UD4B, UD4C, UD5A, UD5B, UD5C, UE2A, UE4A, UE4B, UE4C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

Commit message: R20260918
Parts:
- UC3, UC4, UD2, UD3, UD4, UD5, UE2, UE4, UE5: footprint Package_DIP:DIP-14_W7.62mm_Socket_LongPads -> pong:pong_DIP-14_W7.62mm_Socket_LongPads
Connections:
- net 6V is gone; now on net 8V: UE5.3
Other:
- moved on the sheet: R24, UC3D, UC4C, UD2B, UD3, UD4A, UD4B, UD4C, UD5A, UD5B, UD5C, UE2A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

Commit message: R20260922
Parts:
- R24: footprint (none) -> Resistor_THT:R_Axial_DIN0207_L6.3mm_D2.5mm_P10.16mm_Horizontal
Changed lines of the file:
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@@
 			)
 		)
-		(property "Footprint" ""
+		(property "Footprint" "Resistor_THT:R_Axial_DIN0207_L6.3mm_D2.5mm_P10.16mm_Horizontal"
 			(at 182.626 90.424 90)
 			(hide yes)
