File: SCORECNTR.kicad_sch (KiCad schematic)
At the start: 0 parts

Commit message: R20260915
Other:
- company: (none) -> Atari
- title: (none) -> PONG
Changed lines of the file:
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@@
 	(generator "eeschema")
 	(generator_version "10.0")
-	(paper "A4")
+	(paper "USLetter")
+	(title_block
+		(title "PONG")
+		(company "Atari")
+	)
 )

Commit message: R20260918
Parts:
- added R28, R29: R, symbol Device:R_US
- added SW1: SW_DPDT_x2, symbol Switch:SW_DPDT_x2
- added UC7, UD7: 7490, pong:pong_DIP-14_W7.62mm_Socket_LongPads, symbol 74xx_IEEE:7490
- added UC8: 74LS107, pong:pong_DIP-14_W7.62mm_Socket_LongPads, symbol 74xx:74LS107
- added UD1: 7404, pong:pong_DIP-14_W7.62mm_Socket_LongPads, symbol 74xx_IEEE:7404
- added UD8: 7410, pong:pong_DIP-14_W7.62mm_Socket_LongPads, symbol 74xx_IEEE:7410
- added UE1, UE6: 7400, pong:pong_DIP-14_W7.62mm_Socket_LongPads, symbol 74xx:7400
- added UF5: 7402, pong:pong_DIP-14_W7.62mm_Socket_LongPads, symbol 74xx:7402
- added UH6: 7420, pong:pong_DIP-14_W7.62mm_Socket_LongPads, symbol 74xx_IEEE:7420
Connections:
- new net: UD1.12, UE1.1
- new net: UC7.14 (~{CKA}), UF5.4
- new net: UD7.14 (~{CKA}), UF5.1
- new net: UD7.2 (R0(1)), UD7.3 (R0(2))
- new net: R29.2, UC8.11 (K), UC8.8 (J)
- new net: R28.2, UC8.1 (J), UC8.4 (K)
- new net: SW1.2 (B), UD8.2
- new net: SW1.5 (B), UD8.4
- new net +3.3V: UC7.5 (VCC), UD1.14 (VCC), UD7.5 (VCC), UD8.14 (VCC), UD8.14 (VCC), UH6.14 (VCC)
- new net +5V: R28.1, R29.1
- new net /SCORE2_10: UC8.6 (~{Q})
- new net /STOPG2: UD8.6
- new net GND: UC7.10 (GND), UC7.6 (R9(1)), UC7.7 (R9(2)), UD1.7 (GND), UD7.10 (GND), UD7.6 (R9(1)), UD7.7 (R9(2)), UD8.7 (GND), UD8.7 (GND), UH6.7 (GND)
- new net HBLANK: UE6.10
- new net HVID: UE6.9, UH6.6
- new net L: UF5.5
- new net MISSED: UE1.3, UF5.2, UF5.6
- new net R: UF5.3
- new net SCORE1_1: UC7.1 (~{CKB}), UC7.12 (Q0), UD8.1
- new net SCORE1_10: UC8.3 (Q), UD8.13
- new net SCORE1_2: UC7.9 (Q1)
- new net SCORE1_4: SW1.3 (C), UC7.8 (Q2)
- new net SCORE1_8: UC7.11 (Q3), UC8.12 (C)
- new net SCORE2_1: UD7.1 (~{CKB}), UD7.12 (Q0), UD8.3
- new net SCORE2_10: UC8.5 (Q), UD8.5
- new net SCORE2_2: UD7.9 (Q1)
- new net SCORE2_4: SW1.6 (C), UD7.8 (Q2)
- new net SCORE2_8: UC8.9 (C), UD7.11 (Q3)
- new net SRST: UC7.2 (R0(1)), UC7.3 (R0(2))
- new net /ATTRACT: UE1.2
- new net /HVID: UH6.1, UH6.2, UH6.4, UH6.5
- new net /MISS: UD1.13, UE6.8
- new net /SCORE1_10: UC8.2 (~{Q})
- new net /SRST: UC8.10 (~{R}), UC8.13 (~{R})
- new net /STOPG1: UD8.12

Commit message: R20260922
Parts:
- R28, R29: footprint (none) -> Resistor_THT:R_Axial_DIN0207_L6.3mm_D2.5mm_P10.16mm_Horizontal
Changed lines of the file:
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@@
 			)
 		)
-		(property "Footprint" ""
+		(property "Footprint" "Resistor_THT:R_Axial_DIN0207_L6.3mm_D2.5mm_P10.16mm_Horizontal"
 			(at 114.554 172.974 90)
 			(hide yes)
@@
 			)
 		)
-		(property "Footprint" ""
+		(property "Footprint" "Resistor_THT:R_Axial_DIN0207_L6.3mm_D2.5mm_P10.16mm_Horizontal"
 			(at 115.824 98.044 90)
 			(hide yes)
