File: VSYNC.kicad_sch (KiCad schematic)
At the start: 5 parts

Commit message: Added remainder of sheets
Parts:
- UD8, UD9, UE7, UE8, UE9: footprint Package_DIP:DIP-14_W10.16mm -> Package_DIP:DIP-14_W7.62mm_Socket_LongPads
Changed lines of the file:
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@@
 			)
 		)
-		(property "Footprint" "Package_DIP:DIP-14_W10.16mm"
+		(property "Footprint" "Package_DIP:DIP-14_W7.62mm_Socket_LongPads"
 			(at 128.27 90.17 0)
 			(hide yes)
@@
 			)
 		)
-		(property "Footprint" "Package_DIP:DIP-14_W10.16mm"
+		(property "Footprint" "Package_DIP:DIP-14_W7.62mm_Socket_LongPads"
 			(at 172.72 91.44 0)
 			(hide yes)
@@
 			)
 		)
-		(property "Footprint" "Package_DIP:DIP-14_W10.16mm"
+		(property "Footprint" "Package_DIP:DIP-14_W7.62mm_Socket_LongPads"
 			(at 59.69 90.17 0)
 			(hide yes)
@@
 			)
 		)
-		(property "Footprint" "Package_DIP:DIP-14_W10.16mm"
+		(property "Footprint" "Package_DIP:DIP-14_W7.62mm_Socket_LongPads"
 			(at 200.66 132.08 0)
 			(hide yes)
@@
 			)
 		)
-		(property "Footprint" "Package_DIP:DIP-14_W10.16mm"
+		(property "Footprint" "Package_DIP:DIP-14_W7.62mm_Socket_LongPads"
 			(at 237.49 134.62 0)
 			(hide yes)

Commit message: R20260915
Parts:
- added R16, R17: R, symbol Device:R_US
Connections:
- net 16V: now reaches UE9.1 (~{CKB}), UE9.12 (Q0)
- net GND: now reaches UE9.10 (GND)
- net GND: now also UD8.7 (GND), UE8.10 (GND)
- net 128V: now reaches UD9.9 (C), UE9.11 (Q3)
- net 8V: now reaches UE8.11 (Q3), UE9.14 (~{CKA})
- net +3.3V: now reaches UE9.5 (VCC)
- net +3.3V: now also UD8.14 (VCC), UE8.5 (VCC)
- net 64V: now reaches UE9.8 (Q2)
- net 32V: now reaches UE9.9 (Q1)
- net at UD9.11 (K), UD9.8 (J): now also R16.2
- net 1V: now reaches UD8.11, UE8.1 (~{CKB}), UE8.12 (Q0)
- net 4V: now reaches UD8.10, UE8.8 (Q2)
- net 2V: now reaches UE8.9 (Q1)
- net at UE7.1 (~{R}), UE7.4 (~{S}): now also R17.2
- new net +5V: R16.1, R17.1
- no-connect marks 0 -> 3
Other:
- company: (none) -> Atari
- title: (none) -> PONG
- moved on the sheet: UD8C, UE7A

Commit message: R20260918
Parts:
- UD8, UD9, UE7, UE8, UE9: footprint Package_DIP:DIP-14_W7.62mm_Socket_LongPads -> pong:pong_DIP-14_W7.62mm_Socket_LongPads
Changed lines of the file:
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@@
 			)
 		)
-		(property "Footprint" "Package_DIP:DIP-14_W7.62mm_Socket_LongPads"
+		(property "Footprint" "pong:pong_DIP-14_W7.62mm_Socket_LongPads"
 			(at 128.27 90.17 0)
 			(hide yes)
@@
 			)
 		)
-		(property "Footprint" "Package_DIP:DIP-14_W7.62mm_Socket_LongPads"
+		(property "Footprint" "pong:pong_DIP-14_W7.62mm_Socket_LongPads"
 			(at 172.72 91.44 0)
 			(hide yes)
@@
 			)
 		)
-		(property "Footprint" "Package_DIP:DIP-14_W7.62mm_Socket_LongPads"
+		(property "Footprint" "pong:pong_DIP-14_W7.62mm_Socket_LongPads"
 			(at 59.69 90.17 0)
 			(hide yes)
@@
 			)
 		)
-		(property "Footprint" "Package_DIP:DIP-14_W7.62mm_Socket_LongPads"
+		(property "Footprint" "pong:pong_DIP-14_W7.62mm_Socket_LongPads"
 			(at 203.2 132.08 0)
 			(hide yes)
@@
 			)
 		)
-		(property "Footprint" "Package_DIP:DIP-14_W7.62mm_Socket_LongPads"
+		(property "Footprint" "pong:pong_DIP-14_W7.62mm_Socket_LongPads"
 			(at 236.22 134.62 0)
 			(hide yes)

Commit message: R20260922
Parts:
- R16, R17: footprint (none) -> Resistor_THT:R_Axial_DIN0207_L6.3mm_D2.5mm_P10.16mm_Horizontal
Changed lines of the file:
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@@
 			)
 		)
-		(property "Footprint" ""
+		(property "Footprint" "Resistor_THT:R_Axial_DIN0207_L6.3mm_D2.5mm_P10.16mm_Horizontal"
 			(at 221.996 118.364 90)
 			(hide yes)
@@
 			)
 		)
-		(property "Footprint" ""
+		(property "Footprint" "Resistor_THT:R_Axial_DIN0207_L6.3mm_D2.5mm_P10.16mm_Horizontal"
 			(at 163.576 77.724 90)
 			(hide yes)
