File: BALLH.kicad_sch (KiCad schematic)
At the start: 4 parts

Commit message: Added remainder of sheets
Parts:
- UE1, UG5, UG6, UH6: footprint Package_DIP:DIP-14_W10.16mm -> Package_DIP:DIP-14_W7.62mm_Socket_LongPads
Changed lines of the file:
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@@
 			)
 		)
-		(property "Footprint" "Package_DIP:DIP-14_W10.16mm"
+		(property "Footprint" "Package_DIP:DIP-14_W7.62mm_Socket_LongPads"
 			(at 105.41 69.85 0)
 			(hide yes)
@@
 			)
 		)
-		(property "Footprint" "Package_DIP:DIP-14_W10.16mm"
+		(property "Footprint" "Package_DIP:DIP-14_W7.62mm_Socket_LongPads"
 			(at 115.57 149.86 0)
 			(hide yes)
@@
 			)
 		)
-		(property "Footprint" "Package_DIP:DIP-14_W10.16mm"
+		(property "Footprint" "Package_DIP:DIP-14_W7.62mm_Socket_LongPads"
 			(at 153.67 100.33 0)
 			(hide yes)
@@
 			)
 		)
-		(property "Footprint" "Package_DIP:DIP-14_W10.16mm"
+		(property "Footprint" "Package_DIP:DIP-14_W7.62mm_Socket_LongPads"
 			(at 152.4 144.78 0)
 			(hide yes)

Commit message: R20260915
Other:
- company: (none) -> Atari
- title: (none) -> PONG
Changed lines of the file:
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@@
 	(generator_version "10.0")
 	(paper "A")
+	(title_block
+		(title "PONG")
+		(company "Atari")
+	)
 	(junction
 		(at 133.35 147.32)

Commit message: R20260918
Parts:
- added R26: R, symbol Device:R_US
- UE1, UG5, UG6, UH6: footprint Package_DIP:DIP-14_W7.62mm_Socket_LongPads -> pong:pong_DIP-14_W7.62mm_Socket_LongPads
Connections:
- net +5V: now also R26.1; no longer UG6.11 (K), UG6.8 (J)
- net /CLR: now also UG6.10 (~{R})
- net +3.3V: now reaches UH6.14 (VCC)
- net +3.3V: now also UG5.14 (VCC)
- net GND: now reaches UH6.7 (GND)
- net GND: now also UG5.7 (GND)
- new net: R26.2, UG6.11 (K), UG6.8 (J)
- no-connect marks 0 -> 1
Other:
- note added: "NEED 9316 UNITS"
- moved on the sheet: UE1B

Commit message: R20260922
Parts:
- R26: footprint (none) -> Resistor_THT:R_Axial_DIN0207_L6.3mm_D2.5mm_P10.16mm_Horizontal
Changed lines of the file:
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@@
 			)
 		)
-		(property "Footprint" ""
+		(property "Footprint" "Resistor_THT:R_Axial_DIN0207_L6.3mm_D2.5mm_P10.16mm_Horizontal"
 			(at 101.346 139.954 90)
 			(hide yes)

Commit message: R20260922PM
Parts:
- added R30, R31: R, Resistor_THT:R_Axial_DIN0207_L6.3mm_D2.5mm_P10.16mm_Horizontal, symbol Device:R_US
- added UG7, UH7: 74LS161, pong:pong_DIP-16_W7.62mm_Socket_LongPads, symbol 74xx:74LS161
Connections:
- net +3.3V: now also UG7.16 (VCC), UH7.16 (VCC)
- net +5V: now also R30.1, R31.1
- net GND: now also UG7.3 (D0), UG7.4 (D1), UG7.5 (D2), UG7.8 (GND), UH7.5 (D2), UH7.8 (GND)
- net /CLR: now also UG7.1 (~{MR}), UH7.1 (~{MR})
- net at UG6.9 (C): now also UG5.9, UH6.12, UG7.15 (TC)
- net at UH6.10: now also UH7.11 (Q3)
- net at UH6.9: now also UH7.12 (Q2)
- net at UG5.10: now also UG7.7 (CEP), UH7.15 (TC)
- net at UG5.8: now also UG7.9 (~{PE}), UH7.9 (~{PE})
- new net: R30.2, UG7.10 (CET), UG7.6 (D3)
- new net: R31.2, UH7.6 (D3), UH7.7 (CEP)
- new net Aa: UH7.3 (D0)
- new net Ba: UH7.4 (D1)
- new net CLK: UG7.2 (CP), UH7.2 (CP)
- new net ~HBLANK: UH7.10 (CET)
- no-connect marks 1 -> 7
Other:
- note removed: "NEED 9316 UNITS"
- moved on the sheet: R26, UG5C, UG6B, UH6B
