File: VBALLCTRL.kicad_sch (KiCad schematic)
At the start: 0 parts

Commit message: R20260915
Other:
- company: (none) -> Atari
- title: (none) -> PONG
Changed lines of the file:
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@@
 	(generator "eeschema")
 	(generator_version "10.0")
-	(paper "A4")
+	(paper "USLetter")
+	(title_block
+		(title "PONG")
+		(company "Atari")
+	)
 )

Commit message: R20260918
Parts:
- added R25: R, symbol Device:R_US
- added UA4: 7486, pong:pong_DIP-14_W7.62mm_Socket_LongPads, symbol 74xx_IEEE:7486
- added UA5, UB5: 74LS74, pong:pong_DIP-14_W7.62mm_Socket_LongPads, symbol 74xx:74LS74
- added UB2: 7400, pong:pong_DIP-14_W7.62mm_Socket_LongPads, symbol 74xx:7400
- added UB4: 7483, pong:pong_DIP-16_W7.62mm_Socket_LongPads, symbol 74xx_IEEE:7483
- added UC4: 7410, pong:pong_DIP-14_W7.62mm_Socket_LongPads, symbol 74xx_IEEE:7410
- added UD1: 7404, pong:pong_DIP-14_W7.62mm_Socket_LongPads, symbol 74xx_IEEE:7404
Connections:
- new net: UB4.3 (A3), UC4.1, UC4.13, UC4.2
- new net: UB4.11 (B1), UC4.12
- new net: UA5.1 (~{R}), UA5.13 (~{R}), UB5.1 (~{R}), UD1.6
- new net: UA4.10, UA4.4
- new net: UA4.5, UA5.5 (Q)
- new net: UA4.6, UB4.8 (A2)
- new net: UA5.10 (~{S}), UA5.4 (~{S}), UB5.4 (~{S})
- new net: UA4.9, UA5.9 (Q)
- new net: UA4.8, UB4.10 (A1)
- new net: R25.2, UB4.4 (B3), UB4.7 (B2)
- new net +3.3V: UA4.14 (VCC), UA4.14 (VCC), UB4.5 (VCC), UC4.14 (VCC), UD1.14 (VCC)
- new net +5V: R25.1
- new net A6: UB4.9 (S1)
- new net ATTRACT: UD1.5
- new net B6: UB4.6 (S2)
- new net C6: UB4.2 (S3)
- new net D6: UB4.15 (S4)
- new net GND: UA4.7 (GND), UA4.7 (GND), UB4.1 (A4), UB4.12 (GND), UB4.13 (C0), UB4.16 (B4), UC4.7 (GND), UD1.7 (GND)
- new net HIT: UA5.11 (C), UA5.3 (C), UB2.12, UB2.13, UB5.3 (C)
- no-connect marks 0 -> 3
Other:
- note added: "NEED 7450 ICS"
- note added: "NEED H2A?"

Commit message: R20260922
Parts:
- R25: footprint (none) -> Resistor_THT:R_Axial_DIN0207_L6.3mm_D2.5mm_P10.16mm_Horizontal
Changed lines of the file:
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@@
 			)
 		)
-		(property "Footprint" ""
+		(property "Footprint" "Resistor_THT:R_Axial_DIN0207_L6.3mm_D2.5mm_P10.16mm_Horizontal"
 			(at 173.736 26.924 90)
 			(hide yes)

Commit message: R20260922PM
Parts:
- added UA6, UB6: 7450, pong:pong_DIP-14_W7.62mm_Socket_LongPads, symbol d1:7450
Connections:
- net at UB4.3 (A3), UC4.1, UC4.13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: now also UB6.8
- net at UA4.10, UA4.4: now also UB6.1
- net at UA5.12 (D): now also UA6.8
- net at UA5.2 (D): now also UA6.6
- net at UB5.2 (D): now also UB6.6
- net at UB5.5 (Q): now also UB6.13
- net at UB5.6 (~{Q}): now also UB6.10
- new net 256H: UA6.5, UA6.9, UB6.5
- new net B1: UA6.10
- new net B2: UA6.1
- new net C1: UA6.3
- new net C2: UA6.4
- new net D1: UB6.3
- new net D2: UB6.4
- new net /256H: UA6.13, UA6.2, UB6.2
Other:
- note removed: "NEED 7450 ICS"
