File: pong.kicad_pcb (KiCad board)
At the start: 2 copper layers, 395.7 x 223.9 mm, 61 parts, among them U2 LM317_TO3

Commit message: R20260914
Parts:
- removed UA8: 7493, Package_DIP:DIP-14_W10.16mm
- removed UA9: NE555P, Package_DIP:DIP-8_W7.62mm
- U2: value LM317_TO3 -> LM309_TO3
- UA2, UA4, UB2, UB4, UB7, UB8, UC1, UC2, UC3, UC4, UC7, UC8, UC9, UD1, UD2, UD3, UD4, UD5, UD7, UD8, UD9, UE1, UE2, UE3, UE4, UE5, UE6, UE7, UE8, UE9, UF1, UF2, UF3, UF5, UF6, UF7, UF8, UF9, UG1, UG2, UG3, UG5, UG6, UH1, UH2, UH3, UH4, UH5, UH6: footprint Package_DIP:DIP-14_W10.16mm -> Package_DIP:DIP-14_W7.62mm_Socket_LongPads
- UB9, UF4, UG4: footprint Package_DIP:DIP-8_W7.62mm -> Package_DIP:DIP-8_W7.62mm_Socket_LongPads
- UC5, UC6, UD6: footprint Package_DIP:DIP-16_W10.16mm -> Package_DIP:DIP-16_W7.62mm_Socket_LongPads
Connections:
- D1 pad 1: unconnected-(D1-K-Pad1) -> Net-(D1-K)
- D2 pad 1: unconnected-(D2-K-Pad1) -> Net-(D1-K)
- U2 pad 1: unconnected-(U2-ADJ-Pad1) -> Net-(D1-K)
- U2 pad 2: unconnected-(U2-VI-Pad2) -> +3.3V
- U2 pad 3: unconnected-(U2-VO-Pad3) -> GND
- UA2 pad 14: unconnected-(UA2C-VCC-Pad14) -> +3.3V
- UA2 pad 7: unconnected-(UA2C-GND-Pad7) -> GND
- UA7 pad 1: /PADDLE2/B1 -> (no net)
- UA7 pad 2: Net-(UA8-Q0) -> (no net)
- UA7 pad 4: /PADDLE2/C1 -> (no net)
- UA7 pad 5: /PADDLE2/D1 -> (no net)
- UA7 pad 6: Net-(UA7-Pad6) -> (no net)
- UB2 pad 14: unconnected-(UB2E-VCC-Pad14) -> +3.3V
- UB2 pad 4: unconnected-(UB2-Pad4) -> Net-(UB2-Pad4)
- UB2 pad 7: unconnected-(UB2E-GND-Pad7) -> GND
- UB7 pad 10: /HSYNC -> (no net)
- UB7 pad 11: /VPAD1 -> (no net)
- UB7 pad 12: Net-(UB7-Pad12) -> (no net)
- UB7 pad 13: Net-(UA7-Pad6) -> (no net)
- UB7 pad 14: unconnected-(UB7E-VCC-Pad14) -> +3.3V
- UB7 pad 7: unconnected-(UB7E-GND-Pad7) -> GND
- UB7 pad 8: Net-(UA8-~{CKA}) -> (no net)
- UB7 pad 9: Net-(UA7-Pad6) -> (no net)
- UB9 pad 4: +5V -> +3.3V
- UB9 pad 8: +5V -> +3.3V
- UC1 pad 14: unconnected-(UC1E-VCC-Pad14) -> +3.3V
- UC1 pad 4: unconnected-(UC1-Pad4) -> /ATTRACT
- UC1 pad 7: unconnected-(UC1E-GND-Pad7) -> GND
- UC2 pad 1: unconnected-(UC2A-~{R}-Pad1) -> /HIT
- UC2 pad 14: unconnected-(UC2C-VCC-Pad14) -> +3.3V
- UC2 pad 2: unconnected-(UC2A-D-Pad2) -> Net-(UC2A-D)
- UC2 pad 3: unconnected-(UC2A-C-Pad3) -> VPOS256
- UC2 pad 4: unconnected-(UC2A-~{S}-Pad4) -> Net-(UC2A-D)
- UC2 pad 6: unconnected-(UC2A-~{Q}-Pad6) -> HIT SOUND EN
- UC2 pad 7: unconnected-(UC2C-GND-Pad7) -> GND
- UC3 pad 1: unconnected-(UC3-Pad1) -> HIT SOUND EN
- UC3 pad 10: unconnected-(UC3-Pad10) -> Net-(UG4-OUT)
- UC3 pad 14: unconnected-(UC3E-VCC-Pad14) -> +3.3V
- UC3 pad 2: unconnected-(UC3-Pad2) -> VPOS16
- UC3 pad 3: unconnected-(UC3-Pad3) -> HIT SOUND EN
- UC3 pad 4: unconnected-(UC3-Pad4) -> VPOS32
- UC3 pad 5: unconnected-(UC3-Pad5) -> Net-(UF3A-Q)
- UC3 pad 7: unconnected-(UC3E-GND-Pad7) -> GND
- UC3 pad 8: unconnected-(UC3-Pad8) -> SCORESOUND
- UC3 pad 9: unconnected-(UC3-Pad9) -> 32V
- UC8 pad 14: unconnected-(UC8C-VCC-Pad14) -> +3.3V
- UC8 pad 7: unconnected-(UC8C-GND-Pad7) -> GND
- UC9 pad 1: Net-(UA8-R0(1)) -> (no net)
- UC9 pad 2: Net-(UB7-Pad12) -> (no net)
- UD2 pad 11: unconnected-(UD2-Pad11) -> /VVID
- UD2 pad 12: unconnected-(UD2-Pad12) -> /VVID
- UD2 pad 13: unconnected-(UD2-Pad13) -> /VVID
- UD2 pad 14: unconnected-(UD2E-VCC-Pad14) -> +3.3V
- UD2 pad 7: unconnected-(UD2E-GND-Pad7) -> GND
- UD9 pad 14: unconnected-(UD9C-VCC-Pad14) -> +3.3V
- UD9 pad 7: unconnected-(UD9C-GND-Pad7) -> GND
- UE1 pad 14: unconnected-(UE1E-VCC-Pad14) -> +3.3V
- UE1 pad 7: unconnected-(UE1E-GND-Pad7) -> GND
- UE2 pad 5: unconnected-(UE2-Pad5) -> Net-(UB2-Pad4)
- UE2 pad 6: unconnected-(UE2-Pad6) -> /VVID
- UE6 pad 14: unconnected-(UE6E-VCC-Pad14) -> +3.3V
- UE6 pad 7: unconnected-(UE6E-GND-Pad7) -> GND
- UE7 pad 14: unconnected-(UE7C-VCC-Pad14) -> +3.3V
- UE7 pad 7: unconnected-(UE7C-GND-Pad7) -> GND
- UF3 pad 1: unconnected-(UF3A-J-Pad1) -> VVID
- UF3 pad 10: +5V -> +3.3V
- UF3 pad 12: unconnected-(UF3A-C-Pad12) -> VBLANK
- UF3 pad 13: unconnected-(UF3A-~{R}-Pad13) -> /SERVE
- UF3 pad 14: unconnected-(UF3C-VCC-Pad14) -> +3.3V
- UF3 pad 3: unconnected-(UF3A-Q-Pad3) -> Net-(UF3A-Q)
- UF3 pad 4: unconnected-(UF3A-K-Pad4) -> /VVID
- UF3 pad 7: unconnected-(UF3C-GND-Pad7) -> GND
- UF5 pad 14: unconnected-(UF5E-VCC-Pad14) -> +3.3V
- UF5 pad 7: unconnected-(UF5E-GND-Pad7) -> GND
- UF6 pad 14: unconnected-(UF6C-VCC-Pad14) -> +3.3V
- UF6 pad 7: unconnected-(UF6C-GND-Pad7) -> GND
- UG1 pad 14: unconnected-(UG1E-VCC-Pad14) -> +3.3V
- UG1 pad 7: unconnected-(UG1E-GND-Pad7) -> GND
- UG3 pad 14: unconnected-(UG3E-VCC-Pad14) -> +3.3V
- UG3 pad 7: unconnected-(UG3E-GND-Pad7) -> GND
- UG4 pad 1: unconnected-(UG4-GND-Pad1) -> GND
- UG4 pad 2: unconnected-(UG4-TRIG-Pad2) -> /MISS
- UG4 pad 3: unconnected-(UG4-OUT-Pad3) -> Net-(UG4-OUT)
- UG4 pad 4: unconnected-(UG4-~{RST}-Pad4) -> +3.3V
- UG4 pad 5: unconnected-(UG4-CONT-Pad5) -> Net-(UG4-CONT)
- UG4 pad 6: unconnected-(UG4-THRES-Pad6) -> Net-(UG4-DISCH)
- UG4 pad 7: unconnected-(UG4-DISCH-Pad7) -> Net-(UG4-DISCH)
- UG4 pad 8: unconnected-(UG4-VCC-Pad8) -> +3.3V
- UG6 pad 11: +5V -> +3.3V
- UG6 pad 7: unconnected-(UG6C-GND-Pad7) -> GND
- UG6 pad 8: +5V -> +3.3V
- UH1 pad 14: unconnected-(UH1E-VCC-Pad14) -> +3.3V
- UH1 pad 7: unconnected-(UH1E-GND-Pad7) -> GND
- UH2 pad 14: unconnected-(UH2C-VCC-Pad14) -> +3.3V
- UH2 pad 7: unconnected-(UH2C-GND-Pad7) -> GND
- UH2 pad 8: +5V -> +3.3V
- UH3 pad 14: unconnected-(UH3C-VCC-Pad14) -> +3.3V
- UH3 pad 7: unconnected-(UH3C-GND-Pad7) -> GND
- UH5 pad 14: unconnected-(UH5E-VCC-Pad14) -> +3.3V
- UH5 pad 7: unconnected-(UH5E-GND-Pad7) -> GND
Routing:
- net +3.3V: track 0.00 -> 333.6 mm
- net (no net): track 217.1 -> 540.9 mm
- net GND: track 1057.9 -> 1291.9 mm
- net Net-(UE1-Pad12): track 0.00 -> 82.5 mm
- net Net-(UF1-Q2): track 0.00 -> 48.2 mm
- net Net-(UF1-~{CKA}): track 0.00 -> 25.0 mm
- net Net-(UF1-Q3): track 0.00 -> 22.9 mm
- net VRESET: track 0.00 -> 15.3 mm
- net Net-(UG1-Pad13): track 0.00 -> 14.2 mm
- net Net-(UH1-Pad12): track 0.00 -> 7.62 mm
Other:
- board text added: "PONG SYZYGY"

Commit message: R20260915
Parts:
- added UA8: 7493, Package_DIP:DIP-14_W7.62mm_Socket_LongPads, F.Cu at (263.9, 0.00)
- added UA9: NE555P, Package_DIP:DIP-8_W7.62mm_Socket_LongPads, F.Cu at (297.4, 0.00)
- U2: value LM309_TO3 -> LM309
- UA7: footprint Package_DIP:DIP-14_W10.16mm -> Package_DIP:DIP-14_W7.62mm_Socket_LongPads
Connections:
- net Net-(UD9B-C) renamed /VSYNC/128V
- net Net-(UE8-Q0) renamed /VSYNC/1V
- net Net-(UE8-Q2) renamed /VSYNC/4V
- net Net-(UE8-Q3) renamed /VSYNC/8V
- net Net-(UE9-Q0) renamed /VSYNC/16V
- net Net-(UF6B-C) renamed /HSYNC/128H
- net Net-(UF8-Q0) renamed /HSYNC/1H
- net Net-(UF8-Q1) renamed /HSYNC/2H
- net Net-(UF8-Q2) renamed /HSYNC/4H
- net Net-(UF8-Q3) renamed /HSYNC/8H
- net Net-(UF9-Q0) renamed /HSYNC/16H
- net Net-(UF9-Q2) renamed /HSYNC/64H
- UA4 pad 10: (no net) -> unconnected-(UA4-Pad10)
- UA4 pad 11: (no net) -> Net-(UA4-Pad11)
- UA4 pad 12: (no net) -> /HSYNC
- UA4 pad 13: (no net) -> /VSYNC
- UA4 pad 14: unconnected-(UA4A-VCC-Pad14) -> +3.3V
- UA4 pad 4: (no net) -> unconnected-(UA4-Pad4)
- UA4 pad 5: (no net) -> unconnected-(UA4-Pad5)
- UA4 pad 6: (no net) -> unconnected-(UA4-Pad6)
- UA4 pad 7: unconnected-(UA4A-GND-Pad7) -> GND
- UA4 pad 8: (no net) -> unconnected-(UA4-Pad8)
- UA4 pad 9: (no net) -> unconnected-(UA4-Pad9)
- UA7 pad 1: (no net) -> Net-(UA8-Q0)
- UA7 pad 14: unconnected-(UA7B-VCC-Pad14) -> +3.3V
- UA7 pad 2: (no net) -> Net-(UA8-Q1)
- UA7 pad 4: (no net) -> Net-(UA8-Q2)
- UA7 pad 5: (no net) -> Net-(UA8-Q3)
- UA7 pad 6: (no net) -> Net-(UA7-Pad6)
- UA7 pad 7: unconnected-(UA7B-GND-Pad7) -> GND
- UB2 pad 1: unconnected-(UB2-Pad1) -> /STOPG1
- UB2 pad 2: unconnected-(UB2-Pad2) -> /STOPG2
- UB2 pad 3: unconnected-(UB2-Pad3) -> Net-(UB2-Pad3)
- UB7 pad 10: (no net) -> /HSYNC
- UB7 pad 11: (no net) -> /VPAD2
- UB7 pad 12: (no net) -> Net-(UA7-Pad6)
- UB7 pad 13: (no net) -> Net-(UB7-Pad13)
- UB7 pad 8: (no net) -> Net-(UA8-~{CKA})
- UB7 pad 9: (no net) -> Net-(UA7-Pad6)
- UB8 pad 10: unconnected-(UB8-GND-Pad10) -> GND
- UB8 pad 5: unconnected-(UB8-VCC-Pad5) -> +3.3V
- UB9 pad 1: unconnected-(UB9-GND-Pad1) -> GND
- UC4 pad 14: unconnected-(UC4A-VCC-Pad14) -> +3.3V
- UC4 pad 7: unconnected-(UC4A-GND-Pad7) -> GND
- UC5 pad 16: unconnected-(UC5-VCC-Pad16) -> +3.3V
- UC5 pad 8: unconnected-(UC5-GND-Pad8) -> GND
- UC6 pad 16: unconnected-(UC6-VCC-Pad16) -> +3.3V
- UC6 pad 8: unconnected-(UC6-GND-Pad8) -> GND
- UC9 pad 1: (no net) -> Net-(UA8-R0(1))
- UC9 pad 12: unconnected-(UC9-Pad12) -> /SRST
- UC9 pad 13: unconnected-(UC9-Pad13) -> Net-(UC9-Pad13)
- UC9 pad 14: unconnected-(UC9B-VCC-Pad14) -> +3.3V
- UC9 pad 2: (no net) -> Net-(UB7-Pad13)
- UC9 pad 5: unconnected-(UC9-Pad5) -> /SRST
- UC9 pad 6: unconnected-(UC9-Pad6) -> Net-(UC9-Pad13)
- UC9 pad 7: unconnected-(UC9B-GND-Pad7) -> GND
- UD1 pad 3: unconnected-(UD1-Pad3) -> /ATTRACT
- UD1 pad 4: unconnected-(UD1-Pad4) -> ATTRACT
- UD1 pad 7: unconnected-(UD1A-GND-Pad7) -> GND
- UD2 pad 1: unconnected-(UD2-Pad1) -> /ATTRACT
- UD2 pad 2: unconnected-(UD2-Pad2) -> Net-(UB2-Pad3)
- UD2 pad 3: unconnected-(UD2-Pad3) -> /RUN
- UD3 pad 1: unconnected-(UD3-Pad1) -> Net-(R24-Pad2)
- UD3 pad 14: unconnected-(UD3-VCC-Pad14) -> +3.3V
- UD3 pad 7: unconnected-(UD3-GND-Pad7) -> GND
- UD4 pad 14: unconnected-(UD4A-VCC-Pad14) -> +3.3V
- UD4 pad 7: unconnected-(UD4A-GND-Pad7) -> GND
- UD5 pad 14: unconnected-(UD5A-VCC-Pad14) -> +3.3V
- UD5 pad 7: unconnected-(UD5A-GND-Pad7) -> GND
- UD6 pad 16: unconnected-(UD6-VCC-Pad16) -> +3.3V
- UD6 pad 8: unconnected-(UD6-GND-Pad8) -> GND
- UD8 pad 14: unconnected-(UD8A-VCC-Pad14) -> +3.3V
- UD8 pad 7: unconnected-(UD8A-GND-Pad7) -> GND
- UE2 pad 14: unconnected-(UE2A-VCC-Pad14) -> +3.3V
- UE2 pad 7: unconnected-(UE2A-GND-Pad7) -> GND
- UE3 pad 14: unconnected-(UE3A-VCC-Pad14) -> +3.3V
- UE3 pad 7: unconnected-(UE3A-GND-Pad7) -> GND
- UE4 pad 11: unconnected-(UE4-Pad11) -> Net-(UA4-Pad11)
- UE4 pad 14: unconnected-(UE4A-VCC-Pad14) -> +3.3V
- UE4 pad 7: unconnected-(UE4A-GND-Pad7) -> GND
- UE4 pad 8: unconnected-(UE4-Pad8) -> Net-(D3-K)
- UE4 pad 9: unconnected-(UE4-Pad9) -> Net-(UB2-Pad3)
- UE5 pad 14: unconnected-(UE5A-VCC-Pad14) -> +3.3V
- UE5 pad 7: unconnected-(UE5A-GND-Pad7) -> GND
- UE8 pad 10: unconnected-(UE8-GND-Pad10) -> GND
- UE8 pad 5: unconnected-(UE8-VCC-Pad5) -> +3.3V
- UE8 pad 9: unconnected-(UE8-Q1-Pad9) -> /VSYNC/2V
- UE9 pad 10: unconnected-(UE9-GND-Pad10) -> GND
- UE9 pad 5: unconnected-(UE9-VCC-Pad5) -> +3.3V
- UE9 pad 8: unconnected-(UE9-Q2-Pad8) -> /VSYNC/64V
- UE9 pad 9: unconnected-(UE9-Q1-Pad9) -> /VSYNC/32V
- UF2 pad 14: unconnected-(UF2A-VCC-Pad14) -> +3.3V
- UF2 pad 7: unconnected-(UF2A-GND-Pad7) -> GND
- UF3 pad 10: +3.3V -> Net-(UF3B-~{R})
- UF7 pad 14: unconnected-(UF7-VCC-Pad14) -> +3.3V
- UF7 pad 7: unconnected-(UF7-GND-Pad7) -> GND
- UF8 pad 10: unconnected-(UF8-GND-Pad10) -> GND
- UF8 pad 5: unconnected-(UF8-VCC-Pad5) -> +3.3V
- UF9 pad 10: unconnected-(UF9-GND-Pad10) -> GND
- UF9 pad 5: unconnected-(UF9-VCC-Pad5) -> +3.3V
- UF9 pad 9: unconnected-(UF9-Q1-Pad9) -> /HSYNC/32H
- UG2 pad 1: (no net) -> /VPAD2
- UG2 pad 10: (no net) -> 256H
- UG2 pad 11: (no net) -> /VPAD1
- UG2 pad 12: (no net) -> PAD2
- UG2 pad 13: (no net) -> Net-(UG2-Pad13)
- UG2 pad 14: unconnected-(UG2B-VCC-Pad14) -> +3.3V
- UG2 pad 2: (no net) -> /256H
- UG2 pad 7: unconnected-(UG2B-GND-Pad7) -> GND
- UG2 pad 8: (no net) -> PAD1
- UG2 pad 9: (no net) -> Net-(UG2-Pad13)
- UG3 pad 10: (no net) -> 128H
- UG3 pad 8: (no net) -> Net-(UG2-Pad13)
- UG3 pad 9: (no net) -> Net-(UH3A-~{Q})
- UG5 pad 14: unconnected-(UG5A-VCC-Pad14) -> +3.3V
- UG5 pad 7: unconnected-(UG5A-GND-Pad7) -> GND
- UH3 pad 1: (no net) -> Net-(UH3A-~{R})
- UH3 pad 2: (no net) -> 128H
- UH3 pad 3: (no net) -> 4H
- UH3 pad 4: (no net) -> /ATTRACT
- UH3 pad 5: (no net) -> unconnected-(UH3A-Q-Pad5)
- UH3 pad 6: (no net) -> Net-(UH3A-~{Q})
Routing:
- net GND: track 1291.9 -> 3202.4 mm
- net +3.3V: track 333.6 -> 2193.8 mm
- net (no net): track 540.9 -> 217.1 mm
- net Net-(UA8-R0(1)): track 0.00 -> 86.0 mm
- net 256H: track 0.00 -> 78.7 mm
- net /256V: track 0.00 -> 77.3 mm
- net 128H: track 0.00 -> 76.6 mm
- net Net-(UB2-Pad3): track 0.00 -> 47.9 mm
- net 4V: track 0.00 -> 47.1 mm
- net /ATTRACT: track 0.00 -> 46.9 mm
- net Net-(UA7-Pad6): track 0.00 -> 45.7 mm
- net Net-(UH3B-D): track 0.00 -> 43.1 mm
- net /VSYNC/V RESET: track 0.00 -> 37.4 mm
- net /VSYNC/1V: track 0.00 -> 35.8 mm
- net Net-(UH2B-~{R}): track 0.00 -> 30.8 mm
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
Commit message: R20260918
Parts:
- added D3: 1N914, Diode_THT:D_DO-35_SOD27_P10.16mm_Horizontal, F.Cu at (321.3, 1.02)
- added D4: 1N914, Diode_THT:D_DO-35_SOD27_P10.16mm_Horizontal, F.Cu at (321.2, -23.4)
- added D5: 1N914, Diode_THT:D_DO-35_SOD27_P10.16mm_Horizontal, F.Cu at (321.1, -45.3)
- added UA5: 74LS74, pong:pong_DIP-14_W7.62mm_Socket_LongPads, F.Cu at (163.3, 0.00)
- added UB5: 74LS74, pong:pong_DIP-14_W7.62mm_Socket_LongPads, F.Cu at (163.3, -24.6)
- UA2, UA4, UA7, UA8, UB2, UB7, UB8, UC1, UC2, UC3, UC4, UC7, UC8, UC9, UD1, UD2, UD3, UD4, UD5, UD7, UD8, UD9, UE1, UE2, UE3, UE4, UE5, UE6, UE7, UE8, UE9, UF1, UF2, UF3, UF5, UF6, UF7, UF8, UF9, UG1, UG2, UG3, UG5, UG6, UH1, UH2, UH3, UH4, UH5, UH6: footprint Package_DIP:DIP-14_W7.62mm_Socket_LongPads -> pong:pong_DIP-14_W7.62mm_Socket_LongPads
- UB4: footprint Package_DIP:DIP-14_W7.62mm_Socket_LongPads -> pong:pong_DIP-16_W7.62mm_Socket_LongPads
- UC5, UC6, UD6: footprint Package_DIP:DIP-16_W7.62mm_Socket_LongPads -> pong:pong_DIP-16_W7.62mm_Socket_LongPads
- moved D1 19.3 mm to (424.2, -102.4), turned to 90 degrees
- moved D2 17.9 mm to (418.8, -102.7), turned to 90 degrees
- moved U2 3.87 mm to (361.1, -161.6)
Connections:
- UA4 pad 10: unconnected-(UA4-Pad10) -> Net-(UA4-Pad10)
- UA4 pad 4: unconnected-(UA4-Pad4) -> Net-(UA4-Pad10)
- UA4 pad 5: unconnected-(UA4-Pad5) -> Net-(UA5A-Q)
- UA4 pad 6: unconnected-(UA4-Pad6) -> Net-(UB4-A2)
- UA4 pad 8: unconnected-(UA4-Pad8) -> Net-(UB4-A1)
- UA4 pad 9: unconnected-(UA4-Pad9) -> Net-(UA5B-Q)
- UB2 pad 10: unconnected-(UB2-Pad10) -> Net-(UB2-Pad10)
- UB2 pad 12: unconnected-(UB2-Pad12) -> HIT
- UB2 pad 13: unconnected-(UB2-Pad13) -> HIT
- UB2 pad 8: unconnected-(UB2-Pad8) -> HIT
- UB2 pad 9: unconnected-(UB2-Pad9) -> Net-(UB2-Pad9)
- UB4 pad 1: unconnected-(UB4-A4-Pad1) -> GND
- UB4 pad 10: unconnected-(UB4-A1-Pad10) -> Net-(UB4-A1)
- UB4 pad 11: unconnected-(UB4-B1-Pad11) -> Net-(UB4-B1)
- UB4 pad 12: unconnected-(UB4-GND-Pad12) -> GND
- UB4 pad 13: unconnected-(UB4-C0-Pad13) -> GND
- UB4 pad 2: unconnected-(UB4-S3-Pad2) -> C6
- UB4 pad 3: unconnected-(UB4-A3-Pad3) -> Net-(UB4-A3)
- UB4 pad 4: unconnected-(UB4-B3-Pad4) -> Net-(UB4-B2)
- UB4 pad 5: unconnected-(UB4-VCC-Pad5) -> +3.3V
- UB4 pad 6: unconnected-(UB4-S2-Pad6) -> B6
- UB4 pad 7: unconnected-(UB4-B2-Pad7) -> Net-(UB4-B2)
- UB4 pad 8: unconnected-(UB4-A2-Pad8) -> Net-(UB4-A2)
- UB4 pad 9: unconnected-(UB4-S1-Pad9) -> A6
- UB8 pad 1: unconnected-(UB8-~{CKB}-Pad1) -> Net-(UB8-Q0)
- UB9 pad 6: Net-(UB9-THRES) -> Net-(UB9-DISCH)
- UB9 pad 7: unconnected-(UB9-DISCH-Pad7) -> Net-(UB9-DISCH)
- UC4 pad 1: unconnected-(UC4-Pad1) -> Net-(UB4-A3)
- UC4 pad 12: unconnected-(UC4-Pad12) -> Net-(UB4-B1)
- UC4 pad 13: unconnected-(UC4-Pad13) -> Net-(UB4-A3)
- UC4 pad 2: unconnected-(UC4-Pad2) -> Net-(UB4-A3)
- UC7 pad 1: unconnected-(UC7-~{CKB}-Pad1) -> SCORE1_1
- UC7 pad 10: unconnected-(UC7-GND-Pad10) -> GND
- UC7 pad 11: unconnected-(UC7-Q3-Pad11) -> SCORE1_8
- UC7 pad 12: unconnected-(UC7-Q0-Pad12) -> SCORE1_1
- UC7 pad 14: unconnected-(UC7-~{CKA}-Pad14) -> Net-(UC7-~{CKA})
- UC7 pad 2: unconnected-(UC7-R0(1)-Pad2) -> SRST
- UC7 pad 3: unconnected-(UC7-R0(2)-Pad3) -> SRST
- UC7 pad 5: unconnected-(UC7-VCC-Pad5) -> +3.3V
- UC7 pad 6: unconnected-(UC7-R9(1)-Pad6) -> GND
- UC7 pad 7: unconnected-(UC7-R9(2)-Pad7) -> GND
- UC7 pad 8: unconnected-(UC7-Q2-Pad8) -> SCORE1_4
- UC7 pad 9: unconnected-(UC7-Q1-Pad9) -> SCORE1_2
- UC8 pad 1: unconnected-(UC8A-J-Pad1) -> Net-(UC8A-J)
- UC8 pad 10: unconnected-(UC8B-~{R}-Pad10) -> /SRST
- UC8 pad 11: unconnected-(UC8B-K-Pad11) -> Net-(UC8B-J)
- UC8 pad 12: unconnected-(UC8A-C-Pad12) -> SCORE1_8
- UC8 pad 13: unconnected-(UC8A-~{R}-Pad13) -> /SRST
- UC8 pad 2: unconnected-(UC8A-~{Q}-Pad2) -> /SCORE1_10
- UC8 pad 3: unconnected-(UC8A-Q-Pad3) -> SCORE1_10
- UC8 pad 4: unconnected-(UC8A-K-Pad4) -> Net-(UC8A-J)
- UC8 pad 5: unconnected-(UC8B-Q-Pad5) -> SCORE2_10
- UC8 pad 6: unconnected-(UC8B-~{Q}-Pad6) -> /SCORE2_10
- UC8 pad 8: unconnected-(UC8B-J-Pad8) -> Net-(UC8B-J)
- UC8 pad 9: unconnected-(UC8B-C-Pad9) -> SCORE2_8
- UD1 pad 12: unconnected-(UD1-Pad12) -> Net-(UD1-Pad12)
- UD1 pad 13: unconnected-(UD1-Pad13) -> /SCORECNTR//MISS
- UD1 pad 14: unconnected-(UD1A-VCC-Pad14) -> +3.3V
- UD1 pad 5: unconnected-(UD1-Pad5) -> ATTRACT
- UD1 pad 6: unconnected-(UD1-Pad6) -> Net-(UA5A-~{R})
- UD2 pad 13: /VVID -> VVID
- UD7 pad 1: unconnected-(UD7-~{CKB}-Pad1) -> SCORE2_1
- UD7 pad 10: unconnected-(UD7-GND-Pad10) -> GND
- UD7 pad 11: unconnected-(UD7-Q3-Pad11) -> SCORE2_8
- UD7 pad 12: unconnected-(UD7-Q0-Pad12) -> SCORE2_1
- UD7 pad 14: unconnected-(UD7-~{CKA}-Pad14) -> Net-(UD7-~{CKA})
- UD7 pad 2: unconnected-(UD7-R0(1)-Pad2) -> Net-(UD7-R0(1))
- UD7 pad 3: unconnected-(UD7-R0(2)-Pad3) -> Net-(UD7-R0(1))
- UD7 pad 5: unconnected-(UD7-VCC-Pad5) -> +3.3V
- UD7 pad 6: unconnected-(UD7-R9(1)-Pad6) -> GND
- UD7 pad 7: unconnected-(UD7-R9(2)-Pad7) -> GND
- UD7 pad 8: unconnected-(UD7-Q2-Pad8) -> SCORE2_4
- UD7 pad 9: unconnected-(UD7-Q1-Pad9) -> SCORE2_2
- UD8 pad 1: unconnected-(UD8-Pad1) -> SCORE1_1
- UD8 pad 12: unconnected-(UD8-Pad12) -> /STOPG1
- UD8 pad 13: unconnected-(UD8-Pad13) -> SCORE1_10
- UD8 pad 2: unconnected-(UD8-Pad2) -> Net-(SW1A-B)
- UD8 pad 3: unconnected-(UD8-Pad3) -> SCORE2_1
- UD8 pad 4: unconnected-(UD8-Pad4) -> Net-(SW1B-B)
- UD8 pad 5: unconnected-(UD8-Pad5) -> SCORE2_10
- UD8 pad 6: unconnected-(UD8-Pad6) -> /STOPG2
- UE1 pad 1: unconnected-(UE1-Pad1) -> Net-(UD1-Pad12)
- UE1 pad 2: unconnected-(UE1-Pad2) -> /ATTRACT
- UE1 pad 3: unconnected-(UE1-Pad3) -> MISSED
- UE5 pad 1: unconnected-(UE5-Pad1) -> /RUN
- UE5 pad 13: unconnected-(UE5-Pad13) -> Net-(UF4-OUT)
- UE5 pad 2: unconnected-(UE5-Pad2) -> STOP G
- UE5 pad 3: 6V -> 8V
- UE6 pad 1: unconnected-(UE6-Pad1) -> RST SPEED
- UE6 pad 10: unconnected-(UE6-Pad10) -> HBLANK
- UE6 pad 2: unconnected-(UE6-Pad2) -> RST SPEED
- UE6 pad 3: unconnected-(UE6-Pad3) -> Net-(UF4-TRIG)
- UE6 pad 4: unconnected-(UE6-Pad4) -> /SRST
- UE6 pad 5: unconnected-(UE6-Pad5) -> /MISS
- UE6 pad 6: unconnected-(UE6-Pad6) -> RST SPEED
- UE6 pad 8: unconnected-(UE6-Pad8) -> /SCORECNTR//MISS
- UE6 pad 9: unconnected-(UE6-Pad9) -> /SCORECNTR/HVID
- UF1 pad 10: unconnected-(UF1-GND-Pad10) -> GND
- UF1 pad 5: unconnected-(UF1-VCC-Pad5) -> +3.3V
- UF4 pad 1: unconnected-(UF4-GND-Pad1) -> GND
- UF4 pad 2: unconnected-(UF4-TRIG-Pad2) -> Net-(UF4-TRIG)
- UF4 pad 3: unconnected-(UF4-OUT-Pad3) -> Net-(UF4-OUT)
- UF4 pad 4: unconnected-(UF4-~{RST}-Pad4) -> Net-(UF4-VCC)
- UF4 pad 5: unconnected-(UF4-CONT-Pad5) -> GND
- UF4 pad 6: unconnected-(UF4-THRES-Pad6) -> GND
- UF4 pad 7: unconnected-(UF4-DISCH-Pad7) -> GND
- UF4 pad 8: unconnected-(UF4-VCC-Pad8) -> Net-(UF4-VCC)
- UF5 pad 1: unconnected-(UF5-Pad1) -> Net-(UD7-~{CKA})
- UF5 pad 2: unconnected-(UF5-Pad2) -> MISSED
- UF5 pad 3: unconnected-(UF5-Pad3) -> R
- UF5 pad 4: unconnected-(UF5-Pad4) -> Net-(UC7-~{CKA})
- UF5 pad 5: unconnected-(UF5-Pad5) -> L
- UF5 pad 6: unconnected-(UF5-Pad6) -> MISSED
- UG1 pad 10: unconnected-(UG1-Pad10) -> Net-(UH2A-C)
- UG3 pad 1: unconnected-(UG3-Pad1) -> PAD1
- UG3 pad 11: unconnected-(UG3-Pad11) -> Net-(UB2-Pad10)
- UG3 pad 12: unconnected-(UG3-Pad12) -> Net-(UG3-Pad12)
- UG3 pad 13: unconnected-(UG3-Pad13) -> PAD2
- UG3 pad 2: unconnected-(UG3-Pad2) -> Net-(UG3-Pad12)
- UG3 pad 3: unconnected-(UG3-Pad3) -> Net-(UB2-Pad9)
- UG6 pad 10: unconnected-(UG6B-~{R}-Pad10) -> /CLR
- UG6 pad 11: +3.3V -> Net-(UG6B-J)
- UG6 pad 8: +3.3V -> Net-(UG6B-J)
- UH1 pad 10: unconnected-(UH1-Pad10) -> VRESET
- UH2 pad 8: +3.3V -> Net-(UH2B-J)
- UH6 pad 1: unconnected-(UH6-Pad1) -> /HVID
- UH6 pad 14: unconnected-(UH6A-VCC-Pad14) -> +3.3V
- UH6 pad 2: unconnected-(UH6-Pad2) -> /HVID
- UH6 pad 4: unconnected-(UH6-Pad4) -> /HVID
- UH6 pad 5: unconnected-(UH6-Pad5) -> /HVID
- UH6 pad 6: unconnected-(UH6-Pad6) -> /SCORECNTR/HVID
- UH6 pad 7: unconnected-(UH6A-GND-Pad7) -> GND
Routing:
- net 4V: track 47.1 -> 162.9 mm
- net GND: track 3202.4 -> 3316.5 mm, vias 0 -> 1
- net /HSYNC/128H: track 0.00 -> 102.5 mm
- net Net-(UB7-Pad1): track 0.00 -> 83.7 mm
- net /HSYNC/64H: track 0.00 -> 82.8 mm
- net 16H: track 0.00 -> 78.0 mm
- net Net-(UB7-Pad13): track 0.00 -> 75.3 mm
- net /VSYNC//V RESET: track 0.00 -> 72.9 mm
- net Net-(UG6B-Q): track 0.00 -> 71.9 mm
- net MOVE: track 7.62 -> 78.0 mm
- net Net-(UE2-Pad12): track 0.00 -> 68.7 mm
- net Net-(UH2A-Q): track 0.00 -> 66.5 mm
- net /SCORECNTR/HVID: track 0.00 -> 59.2 mm
- net Net-(UH2A-J): track 11.5 -> 69.8 mm
- net /SCORE1_10: track 23.9 -> 81.5 mm
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
Commit message: R20260921
Parts:
- added C13: C_US, Capacitor_THT:C_Disc_D16.0mm_W5.0mm_P10.00mm, F.Cu at (31.8, -186.9)
- added C14: C_US, Capacitor_THT:C_Disc_D16.0mm_W5.0mm_P10.00mm, F.Cu at (65.4, -186.9)
- added C15: C_US, Capacitor_THT:C_Disc_D16.0mm_W5.0mm_P10.00mm, F.Cu at (98.9, -186.9)
- added C16: C_US, Capacitor_THT:C_Disc_D16.0mm_W5.0mm_P10.00mm, F.Cu at (132.4, -186.9)
- added C17: C_US, Capacitor_THT:C_Disc_D16.0mm_W5.0mm_P10.00mm, F.Cu at (165.9, -186.9)
- added C18: C_US, Capacitor_THT:C_Disc_D16.0mm_W5.0mm_P10.00mm, F.Cu at (199.5, -186.9)
- added C19: C_US, Capacitor_THT:C_Disc_D16.0mm_W5.0mm_P10.00mm, F.Cu at (233.0, -186.9)
- added C20: C_US, Capacitor_THT:C_Disc_D16.0mm_W5.0mm_P10.00mm, F.Cu at (266.5, -186.9)
- added C21: C_US, Capacitor_THT:C_Disc_D16.0mm_W5.0mm_P10.00mm, F.Cu at (300.1, -186.9)
Connections:
- UA5 pad 14: unconnected-(UA5C-VCC-Pad14) -> +3.3V
- UA5 pad 7: unconnected-(UA5C-GND-Pad7) -> GND
- UB5 pad 14: unconnected-(UB5C-VCC-Pad14) -> +3.3V
- UB5 pad 7: unconnected-(UB5C-GND-Pad7) -> GND
- UD1 pad 10: unconnected-(UD1-Pad10) -> (no net)
- UD1 pad 11: unconnected-(UD1-Pad11) -> (no net)
- UD1 pad 8: unconnected-(UD1-Pad8) -> (no net)
- UD1 pad 9: unconnected-(UD1-Pad9) -> (no net)
- UD9 pad 1: unconnected-(UD9A-J-Pad1) -> (no net)
- UD9 pad 12: unconnected-(UD9A-C-Pad12) -> (no net)
- UD9 pad 13: unconnected-(UD9A-~{R}-Pad13) -> (no net)
- UD9 pad 2: unconnected-(UD9A-~{Q}-Pad2) -> (no net)
- UD9 pad 3: unconnected-(UD9A-Q-Pad3) -> (no net)
- UD9 pad 4: unconnected-(UD9A-K-Pad4) -> (no net)
- UE7 pad 8: /HSYNC/H RESET -> HRESET
- UF8 pad 2: /HSYNC/H RESET -> HRESET
- UF8 pad 3: /HSYNC/H RESET -> HRESET
- UF9 pad 2: /HSYNC/H RESET -> HRESET
- UF9 pad 3: /HSYNC/H RESET -> HRESET
- UH4 pad 14: unconnected-(UH4E-VCC-Pad14) -> +3.3V
- UH4 pad 7: unconnected-(UH4E-GND-Pad7) -> GND
Routing:
- net +3.3V: track 2241.8 -> 2333.7 mm
- net HRESET: track 0.00 -> 85.5 mm
- net (no net): track 181.1 -> 246.6 mm, vias 0 -> 4
- net Net-(UG2-Pad5): track 0.00 -> 39.9 mm
- net /HSYNC/H RESET: track 38.4 -> 0.00 mm
- net SCORE2_2: track 0.00 -> 33.8 mm, vias 0 -> 1
- net /STOPG1: track 0.00 -> 31.8 mm, vias 0 -> 1
- net /STOPG2: track 0.00 -> 30.6 mm, vias 0 -> 1
- net Net-(UB2-Pad3): track 47.9 -> 77.2 mm, vias 0 -> 1
- net Net-(UB4-A2): track 0.00 -> 26.7 mm
- net Net-(UB4-A1): track 0.00 -> 25.7 mm
- net Net-(UB8-R0(1)): track 39.8 -> 62.6 mm
- net GND: track 3316.5 -> 3332.1 mm
- net /SCORE2_10: track 23.9 -> 38.1 mm, vias 0 -> 1
- net /SCORE2/scoreBC: track 0.00 -> 11.2 mm, vias 0 -> 1
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