File: pong.kicad_pcb (KiCad board)
At the start: 2 copper layers, 395.7 x 223.9 mm, 75 parts, among them U2 LM309

Commit message: R20260922
Parts:
- added C1: 100pF, Capacitor_THT:C_Disc_D10.5mm_W5.0mm_P7.50mm, F.Cu at (333.2, -68.6)
- added C10: C, Capacitor_THT:C_Axial_L3.8mm_D2.6mm_P10.00mm_Horizontal, F.Cu at (333.5, -55.5)
- added C11: .1, Capacitor_THT:C_Axial_L3.8mm_D2.6mm_P10.00mm_Horizontal, F.Cu at (310.4, -10.2)
- added C12: .1, Capacitor_THT:C_Axial_L3.8mm_D2.6mm_P10.00mm_Horizontal, F.Cu at (340.6, -8.86)
- added C2: .1uF, Capacitor_THT:C_Disc_D10.5mm_W5.0mm_P7.50mm, F.Cu at (329.3, -76.1)
- added C7: C, Capacitor_THT:C_Disc_D16.0mm_W5.0mm_P10.00mm, F.Cu at (364.9, 44.9)
- added C8: .1uF, Capacitor_THT:C_Axial_L3.8mm_D2.6mm_P12.50mm_Horizontal, F.Cu at (310.3, -21.9)
- added C9: .1uF, Capacitor_THT:C_Axial_L3.8mm_D2.6mm_P10.00mm_Horizontal, F.Cu at (345.4, -33.5)
- added D6: 1N914, Diode_THT:D_DO-35_SOD27_P10.16mm_Horizontal, F.Cu at (321.2, 1.14)
- added D7: 1N914, Diode_THT:D_DO-35_SOD27_P10.16mm_Horizontal, F.Cu at (321.4, -23.4)
- added R1: 330, Resistor_THT:R_Axial_DIN0207_L6.3mm_D2.5mm_P10.16mm_Horizontal, F.Cu at (321.2, -67.1)
- added R10: 56K, Resistor_THT:R_Axial_DIN0207_L6.3mm_D2.5mm_P10.16mm_Horizontal, F.Cu at (325.3, -23.4)
- added R11: R, Resistor_THT:R_Axial_DIN0207_L6.3mm_D2.5mm_P10.16mm_Horizontal, F.Cu at (340.6, -33.7)
- added R12: 330, Resistor_THT:R_Axial_DIN0207_L6.3mm_D2.5mm_P10.16mm_Horizontal, F.Cu at (325.2, -55.2)
- added R13: 100, Resistor_THT:R_Axial_DIN0207_L6.3mm_D2.5mm_P10.16mm_Horizontal, F.Cu at (329.2, -55.5)
- added R14: R, Resistor_THT:R_Axial_DIN0207_L6.3mm_D2.5mm_P10.16mm_Horizontal, F.Cu at (445.0, -6.86)
- added R15: R, Resistor_THT:R_Axial_DIN0207_L6.3mm_D2.5mm_P10.16mm_Horizontal, F.Cu at (445.0, -2.81)
- added R16: R, Resistor_THT:R_Axial_DIN0207_L6.3mm_D2.5mm_P10.16mm_Horizontal, F.Cu at (429.7, 3.24)
- added R17: R, Resistor_THT:R_Axial_DIN0207_L6.3mm_D2.5mm_P10.16mm_Horizontal, F.Cu at (429.7, 7.29)
- added R18: R, Resistor_THT:R_Axial_DIN0207_L6.3mm_D2.5mm_P10.16mm_Horizontal, F.Cu at (429.7, 25.4)
- added R19: R, Resistor_THT:R_Axial_DIN0207_L6.3mm_D2.5mm_P10.16mm_Horizontal, F.Cu at (429.7, 13.3)
- added R2: 330, Resistor_THT:R_Axial_DIN0207_L6.3mm_D2.5mm_P10.16mm_Horizontal, F.Cu at (325.4, -67.3)
- added R20: 470, Resistor_THT:R_Axial_DIN0207_L6.3mm_D2.5mm_P10.16mm_Horizontal, F.Cu at (345.4, -9.02)
- added R21: 56K, Resistor_THT:R_Axial_DIN0207_L6.3mm_D2.5mm_P10.16mm_Horizontal, F.Cu at (325.2, 1.14)
- added R22: R, Resistor_THT:R_Axial_DIN0207_L6.3mm_D2.5mm_P10.16mm_Horizontal, F.Cu at (429.7, -6.86)
- added R23: R, Resistor_THT:R_Axial_DIN0207_L6.3mm_D2.5mm_P10.16mm_Horizontal, F.Cu at (429.7, -2.81)
- added R24: R, Resistor_THT:R_Axial_DIN0207_L6.3mm_D2.5mm_P10.16mm_Horizontal, F.Cu at (445.0, 19.4)
- added R25: R, Resistor_THT:R_Axial_DIN0207_L6.3mm_D2.5mm_P10.16mm_Horizontal, F.Cu at (445.0, 25.4)
- added R26: R, Resistor_THT:R_Axial_DIN0207_L6.3mm_D2.5mm_P10.16mm_Horizontal, F.Cu at (445.0, 13.3)
- added R27: R, Resistor_THT:R_Axial_DIN0207_L6.3mm_D2.5mm_P10.16mm_Horizontal, F.Cu at (429.7, 19.4)
- added R28: R, Resistor_THT:R_Axial_DIN0207_L6.3mm_D2.5mm_P10.16mm_Horizontal, F.Cu at (445.0, 3.24)
- added R29: R, Resistor_THT:R_Axial_DIN0207_L6.3mm_D2.5mm_P10.16mm_Horizontal, F.Cu at (445.0, 7.29)
- added R3: 1K, Resistor_THT:R_Axial_DIN0207_L6.3mm_D2.5mm_P10.16mm_Horizontal, F.Cu at (327.6, 51.5)
- added R4: 22K, Resistor_THT:R_Axial_DIN0207_L6.3mm_D2.5mm_P10.16mm_Horizontal, F.Cu at (327.6, 55.6)
- added R5: 1.2, Resistor_THT:R_Axial_DIN0207_L6.3mm_D2.5mm_P10.16mm_Horizontal, F.Cu at (327.6, 59.6)
- added R6: R, Resistor_THT:R_Axial_DIN0207_L6.3mm_D2.5mm_P10.16mm_Horizontal, F.Cu at (429.7, 31.5)
- added R7: 220K, Resistor_THT:R_Axial_DIN0207_L6.3mm_D2.5mm_P10.16mm_Horizontal, F.Cu at (342.9, 53.5)
- added R8: 100, Resistor_THT:R_Axial_DIN0207_L6.3mm_D2.5mm_P10.16mm_Horizontal, F.Cu at (327.6, 33.3)
- added R9: 220, Resistor_THT:R_Axial_DIN0207_L6.3mm_D2.5mm_P10.16mm_Horizontal, F.Cu at (327.6, 37.4)
- added RV1: R_Potentiometer_US, Potentiometer_THT:Potentiometer_Bourns_3296Y_Vertical, F.Cu at (330.3, -9.02)
- added Y1: 14.318Mhz, Crystal:Crystal_HC49-U_Vertical, F.Cu at (338.3, -74.3)
- D5: value 1N914 -> 1N4001; footprint Diode_THT:D_DO-35_SOD27_P10.16mm_Horizontal -> Diode_THT:D_DO-41_SOD81_P10.16mm_Horizontal
- moved D5 73.3 mm to (309.6, 27.1), turned to -90 degrees
- moved D3 50.5 mm to (285.6, 36.7)
- moved D4 21.8 mm to (321.3, -45.2)
Connections:
- UA9 pad 6: Net-(UA9-DISCH) -> Net-(D6-A)
- UA9 pad 7: Net-(UA9-DISCH) -> Net-(D6-K)
- UB9 pad 6: Net-(UB9-DISCH) -> Net-(D7-A)
- UB9 pad 7: Net-(UB9-DISCH) -> Net-(D7-K)
Routing:
- net Net-(R1-Pad2): track 0.00 -> 50.9 mm
- net Net-(C2-Pad1): track 0.00 -> 35.6 mm
- net Net-(C1-Pad1): track 0.00 -> 29.6 mm
- net Net-(C2-Pad2): track 2.54 -> 31.1 mm
- net Net-(D6-A): track 0.00 -> 25.2 mm
- net Net-(D7-K): track 0.00 -> 25.1 mm
- net Net-(D6-K): track 0.00 -> 24.9 mm
- net Net-(D7-A): track 0.00 -> 24.0 mm
- net GND: track 3332.1 -> 3351.1 mm, vias 1 -> 2
- net /SRST: track 49.3 -> 64.6 mm
- net Net-(C1-Pad2): track 0.00 -> 8.74 mm
- net Net-(C10-Pad2): track 0.00 -> 4.08 mm
- net /RUN: track 0.00 -> 3.99 mm

Commit message: R20260922PM
Parts:
- added C6: 1.0, Capacitor_THT:C_Axial_L3.8mm_D2.6mm_P10.00mm_Horizontal, F.Cu at (144.3, -144.1)
- added R30: R, Resistor_THT:R_Axial_DIN0207_L6.3mm_D2.5mm_P10.16mm_Horizontal, F.Cu at (451.2, 46.1)
- added R31: R, Resistor_THT:R_Axial_DIN0207_L6.3mm_D2.5mm_P10.16mm_Horizontal, F.Cu at (451.2, 50.2)
- added UA3: 74LS161, pong:pong_DIP-16_W7.62mm_Socket_LongPads, F.Cu at (96.3, 0.00)
- added UA6: 7450, pong:pong_DIP-14_W7.62mm_Socket_LongPads, F.Cu at (196.8, 0.00)
- added UB3: 74LS161, pong:pong_DIP-16_W7.62mm_Socket_LongPads, F.Cu at (96.3, -24.6)
- added UB6: 7450, pong:pong_DIP-14_W7.62mm_Socket_LongPads, F.Cu at (196.8, -24.6)
- added UG7: 74LS161, pong:pong_DIP-16_W7.62mm_Socket_LongPads, F.Cu at (230.4, -134.1)
- added UH7: 74LS161, pong:pong_DIP-16_W7.62mm_Socket_LongPads, F.Cu at (230.4, -156.0)
- C10: value C -> .1
- C7: value C -> .1; footprint Capacitor_THT:C_Disc_D16.0mm_W5.0mm_P10.00mm -> Capacitor_THT:C_Axial_L3.8mm_D2.6mm_P10.00mm_Horizontal
- moved C7 291.6 mm to (141.4, -142.3), turned to -90 degrees
- moved R7 287.3 mm to (124.3, -133.0), turned to 90 degrees
Connections:
- R8 pad 1: unconnected-(R8-Pad1) -> Net-(Q1-E)
- UA5 pad 12: unconnected-(UA5B-D-Pad12) -> Net-(UA5B-D)
- UA5 pad 2: unconnected-(UA5A-D-Pad2) -> Net-(UA5A-D)
- UB2 pad 5: unconnected-(UB2-Pad5) -> Net-(UA3-CEP)
- UB2 pad 6: unconnected-(UB2-Pad6) -> Net-(UA3-~{PE})
- UB5 pad 2: unconnected-(UB5A-D-Pad2) -> Net-(UB5A-D)
- UB5 pad 5: unconnected-(UB5A-Q-Pad5) -> Net-(UB5A-Q)
- UB5 pad 6: unconnected-(UB5A-~{Q}-Pad6) -> Net-(UB5A-~{Q})
- UE2 pad 3: unconnected-(UE2-Pad3) -> Net-(UB3-Q2)
- UE2 pad 4: unconnected-(UE2-Pad4) -> Net-(UB3-Q3)
- UG5 pad 10: unconnected-(UG5-Pad10) -> Net-(UG7-CEP)
- UG5 pad 8: unconnected-(UG5-Pad8) -> Net-(UG7-~{PE})
- UG5 pad 9: Net-(UG5-Pad9) -> Net-(UG6B-C)
- UG6 pad 9: unconnected-(UG6B-C-Pad9) -> Net-(UG6B-C)
- UH6 pad 10: unconnected-(UH6-Pad10) -> Net-(UH7-Q3)
- UH6 pad 12: Net-(UG5-Pad9) -> Net-(UG6B-C)
- UH6 pad 9: unconnected-(UH6-Pad9) -> Net-(UH7-Q2)
Routing:
- net Net-(UB4-A3): track 33.1 -> 115.2 mm
- net /HSYNC: track 0.00 -> 64.9 mm
- net Net-(UB5A-D): track 0.00 -> 48.0 mm
- net Net-(UA3-CET): track 0.00 -> 42.7 mm
- net GND: track 3351.1 -> 3391.4 mm
- net Net-(UB5A-~{Q}): track 0.00 -> 34.1 mm
- net Net-(UB5A-Q): track 0.00 -> 29.7 mm
- net 256H: track 112.8 -> 139.6 mm
- net Net-(UA3-~{PE}): track 0.00 -> 25.7 mm
- net /256H: track 0.00 -> 24.6 mm
- net /CLR: track 0.00 -> 22.4 mm
- net CLK: track 0.00 -> 22.4 mm
- net +3.3V: track 2333.7 -> 2351.0 mm
- net unconnected-(UG5-Pad8): track 10.9 -> 0.00 mm, vias 1 -> 0
- net Net-(UG7-~{PE}): track 0.00 -> 10.9 mm, vias 0 -> 1
