File: pong.kicad_pcb (KiCad board)
At the start: 2 copper layers, 395.7 x 223.9 mm, 125 parts, among them U2 LM309, Y1 14.318Mhz

Commit message: R20260924
Parts:
- added C22: .1, Capacitor_THT:C_Axial_L3.8mm_D2.6mm_P10.00mm_Horizontal, F.Cu at (353.2, -55.2)
- added C23: 4.7, Capacitor_THT:C_Axial_L3.8mm_D2.6mm_P10.00mm_Horizontal, F.Cu at (243.4, 46.6)
- added C24: .1, Capacitor_THT:C_Axial_L3.8mm_D2.6mm_P10.00mm_Horizontal, F.Cu at (270.9, 41.0)
- added D8: 1N914, Diode_THT:D_DO-35_SOD27_P10.16mm_Horizontal, F.Cu at (321.2, -88.8)
- added R32: 100, Resistor_THT:R_Axial_DIN0207_L6.3mm_D2.5mm_P10.16mm_Horizontal, F.Cu at (349.2, -45.3)
- added R33: 330k, Resistor_THT:R_Axial_DIN0207_L6.3mm_D2.5mm_P10.16mm_Horizontal, F.Cu at (124.6, -121.3)
- R5: value 1.2 -> 1.2K
- moved R4 257.8 mm to (121.4, -99.2), turned to -90 degrees
- moved R3 252.9 mm to (124.5, -99.2), turned to -90 degrees
- moved R5 244.8 mm to (124.6, -77.1), turned to -90 degrees
- moved R8 90.9 mm to (345.6, -55.8), turned to -90 degrees
- moved R9 64.6 mm to (349.1, -23.5), turned to 90 degrees
- moved C9 11.9 mm to (340.7, -22.6), turned to 90 degrees
- moved R11 11.4 mm to (345.4, -23.4), turned to 90 degrees
Connections:
- R9 pad 1: unconnected-(R9-Pad1) -> Net-(Q2-B)
- UF4 pad 4: Net-(UF4-VCC) -> +3.3V
- UF4 pad 5: GND -> Net-(UF4-CONT)
- UF4 pad 6: GND -> Net-(UF4-CONT)
- UF4 pad 7: GND -> Net-(UF4-CONT)
- UF4 pad 8: Net-(UF4-VCC) -> +3.3V
Routing:
- net VIDEO: track 0.00 -> 11.7 mm
- net Net-(UF4-VCC): track 10.8 -> 0.00 mm
- net +3.3V: track 2351.0 -> 2361.8 mm
- net GND: track 3391.4 -> 3395.2 mm
- net Net-(UF4-CONT): track 0.00 -> 2.54 mm
- net Net-(UB7-Pad13): track 75.3 -> 76.8 mm
- net /SRST: track 64.6 -> 65.8 mm
- net Net-(C2-Pad2): track 31.1 -> 31.7 mm
