File: pong.kicad_sch (KiCad schematic)
At the start: 41 parts, among them U1 L7805, U2 LM317_TO3

Commit message: Added remainder of sheets
Parts:
- removed D1, D2: 1N4001, Diode_THT:D_DO-41_SOD81_P10.16mm_Horizontal, symbol Diode:1N4001
- removed U2: LM317_TO3, Package_TO_SOT_THT:TO-3, symbol Regulator_Linear:LM317_TO3
- removed unit 3 of UA2
- removed unit 5 of UB2
- removed unit 2 of UB2
- removed UB7, UC3, UH1, UH5: 7400, Package_DIP:DIP-14_W10.16mm, symbol 74xx:7400
- removed unit 2 of UC1
- removed unit 5 of UC1
- removed unit 1 of UC2
- removed unit 3 of UC2
- removed unit 3 of UC8
- removed unit 4 of UD2
- removed unit 5 of UD2
- removed unit 3 of UD9
- removed unit 5 of UE1
- removed UE2: 7410, Package_DIP:DIP-14_W10.16mm, symbol 74xx_IEEE:7410
- removed unit 5 of UE6
- removed UE7, UH3: 74LS74, Package_DIP:DIP-14_W10.16mm, symbol 74xx:74LS74
- removed UF3, UF6, UH2: 74LS107, Package_DIP:DIP-14_W10.16mm, symbol 74xx:74LS107
- removed unit 5 of UF5
- removed UG1: 7402, Package_DIP:DIP-14_W10.16mm, symbol 74xx:7402
- removed unit 5 of UG3
- removed UG4: NE555P, Package_DIP:DIP-8_W7.62mm, symbol Timer:NE555P
- removed unit 3 of UG6
- UA2, UA4, UB2, UB4, UC1, UC2, UC4, UC7, UC8, UC9, UD1, UD2, UD7, UD8, UD9, UE1, UE4, UE5, UE6, UF5, UG3, UG6, UH4, UH6: footprint Package_DIP:DIP-14_W10.16mm -> Package_DIP:DIP-14_W7.62mm_Socket_LongPads
- UF4: footprint Package_DIP:DIP-8_W7.62mm -> Package_DIP:DIP-8_W7.62mm_Socket_LongPads
Other:
- added sheet GAMECTRL (GAMECTRL.kicad_sch)
- added sheet POWER (POWER.kicad_sch)
- added sheet SCORECNTR (SCORECNTR.kicad_sch)
- added sheet SOUND (SOUND.kicad_sch)
- added sheet VBALLCNTR (BALLV.kicad_sch)
- added sheet VBALLCTRL (VBALLCTRL.kicad_sch)

Commit message: R20260915
Parts:
- removed unit 3 of UB2
- removed unit 1 of UB2
- removed UC9, UE4: 7404, Package_DIP:DIP-14_W7.62mm_Socket_LongPads, symbol 74xx_IEEE:7404
- removed unit 2 of UD1
- removed UD2: 7402, Package_DIP:DIP-14_W7.62mm_Socket_LongPads, symbol 74xx:7402
- removed UE5: 7427, Package_DIP:DIP-14_W7.62mm_Socket_LongPads, symbol 74xx_IEEE:7427
- removed unit 2 of UE6
- removed unit 1 of UE6
- removed UF4: NE555P, Package_DIP:DIP-8_W7.62mm_Socket_LongPads, symbol Timer:NE555P
- removed UG3: 7400, Package_DIP:DIP-14_W7.62mm_Socket_LongPads, symbol 74xx:7400
- added unit 2 of UA4
- added unit 3 of UA4
Other:
- company: (none) -> Atari
- title: (none) -> PONG
- moved on the sheet: U1, UB4, UC1A, UC1C, UC2B, UC4A, UC4B, UC7, UC8A, UC8B, UD1C, UD1D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

Commit message: R20260918
Parts:
- removed unit 2 of UA4
- removed unit 3 of UA4
- removed UB2, UE1, UE6: 7400, Package_DIP:DIP-14_W7.62mm_Socket_LongPads, symbol 74xx:7400
- removed UB4: 7483, Package_DIP:DIP-14_W7.62mm_Socket_LongPads, symbol 74xx_IEEE:7483
- removed unit 1 of UC4
- removed UC7, UD7: 7490, Package_DIP:DIP-14_W7.62mm_Socket_LongPads, symbol 74xx_IEEE:7490
- removed UC8: 74LS107, Package_DIP:DIP-14_W7.62mm_Socket_LongPads, symbol 74xx:74LS107
- removed unit 6 of UD1
- removed unit 3 of UD1
- removed UD8: 7410, Package_DIP:DIP-14_W7.62mm_Socket_LongPads, symbol 74xx_IEEE:7410
- removed UF5: 7402, Package_DIP:DIP-14_W7.62mm_Socket_LongPads, symbol 74xx:7402
- removed UH6: 7420, Package_DIP:DIP-14_W7.62mm_Socket_LongPads, symbol 74xx_IEEE:7420
- added UB5: 74LS74, pong:pong_DIP-14_W7.62mm_Socket_LongPads, symbol 74xx:74LS74
- UA2, UA4, UC1, UC2, UC4, UD1, UD9, UG6, UH4: footprint Package_DIP:DIP-14_W7.62mm_Socket_LongPads -> pong:pong_DIP-14_W7.62mm_Socket_LongPads

Commit message: R20260921
Parts:
- removed UD1: 7404, pong:pong_DIP-14_W7.62mm_Socket_LongPads, symbol 74xx_IEEE:7404
- removed UD9: 74LS107, pong:pong_DIP-14_W7.62mm_Socket_LongPads, symbol 74xx:74LS107
- removed UH4: 7400, pong:pong_DIP-14_W7.62mm_Socket_LongPads, symbol 74xx:7400

Commit message: R20260922PM
Other:
- moved on the sheet: UA4A, UC4B
Changed lines of the file:
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@@
 	(symbol
 		(lib_id "74xx_IEEE:7410")
-		(at 321.31 -163.83 0)
+		(at 410.21 -166.37 0)
 		(unit 2)
 		(body_style 1)
@@
 		(fields_autoplaced yes)
 		(property "Reference" "UC4"
-			(at 330.2 -170.2502 0)
+			(at 419.1 -172.7902 0)
 			(show_name no)
 			(do_not_autoplace no)
@@
 		)
 		(property "Value" "7410"
-			(at 330.2 -167.7102 0)
+			(at 419.1 -170.2502 0)
 			(show_name no)
 			(do_not_autoplace no)
@@
 		)
 		(property "Footprint" "pong:pong_DIP-14_W7.62mm_Socket_LongPads"
-			(at 321.31 -163.83 0)
+			(at 410.21 -166.37 0)
 			(hide yes)
 			(show_name no)
@@
 		)
 		(property "Datasheet" ""
-			(at 321.31 -163.83 0)
+			(at 410.21 -166.37 0)
 			(hide yes)
 			(show_name no)
@@
 		)
 		(property "Description" ""
-			(at 321.31 -163.83 0)
+			(at 410.21 -166.37 0)
 			(hide yes)
 			(show_name no)
@@
 	(symbol
 		(lib_id "74xx_IEEE:7486")
-		(at 298.45 -52.07 0)
+		(at 387.35 -54.61 0)
 		(unit 1)
 		(body_style 1)
@@
 		(fields_autoplaced yes)
 		(property "Reference" "UA4"
-			(at 307.34 -58.4902 0)
+			(at 396.24 -61.0302 0)
 			(show_name no)
 			(do_not_autoplace no)
@@
 		)
 		(property "Value" "7486"
-			(at 307.34 -55.9502 0)
+			(at 396.24 -58.4902 0)
 			(show_name no)
 			(do_not_autoplace no)
@@
 		)
 		(property "Footprint" "pong:pong_DIP-14_W7.62mm_Socket_LongPads"
-			(at 298.45 -52.07 0)
+			(at 387.35 -54.61 0)
 			(hide yes)
 			(show_name no)
@@
 		)
 		(property "Datasheet" ""
-			(at 298.45 -52.07 0)
+			(at 387.35 -54.61 0)
 			(hide yes)
 			(show_name no)
@@
 		)
 		(property "Description" ""
-			(at 298.45 -52.07 0)
-			(hide yes)
-			(show_name no)
+			(at 387.35 -54.61 0)
+			(hide yes)
+			(show_name no)
