File: GAMECTRL.kicad_sch (KiCad schematic)
At the start: 0 parts

Commit message: R20260915
Parts:
- added C10: C, symbol Device:C
- added D3, D4, D5: 1N914, symbol Device:D
- added R12: 330, symbol Device:R_US
- added R13, R8: 100, symbol Device:R_US
- added R9: 220, symbol Device:R_US
- added SW1: COIN SW, symbol Switch:SW_SPDT
- added UB2, UE6, UG3: 7400, Package_DIP:DIP-14_W7.62mm_Socket_LongPads, symbol 74xx:7400
- added UC9, UD1, UE4: 7404, Package_DIP:DIP-14_W7.62mm_Socket_LongPads, symbol 74xx_IEEE:7404
- added UD2: 7402, Package_DIP:DIP-14_W7.62mm_Socket_LongPads, symbol 74xx:7402
- added UE5: 7427, Package_DIP:DIP-14_W7.62mm_Socket_LongPads, symbol 74xx_IEEE:7427
- added UF4: NE555P, Package_DIP:DIP-8_W7.62mm_Socket_LongPads, symbol Timer:NE555P
Connections:
- new net: D3.2 (A), R8.2, R9.2
- new net: UB2.3, UD2.2, UE4.9
- new net: D3.1 (K), UE4.8
- new net: C10.2, R12.2, R13.2
- new net: SW1.1 (A), UC9.13, UC9.6
- new net +5V: UC9.14 (VCC), UC9.14 (VCC)
- new net ATTRACT: UD1.4
- new net GND: C10.1, D5.1 (K), R13.1, SW1.2 (B), UC9.7 (GND), UC9.7 (GND), UD1.7 (GND), UE4.7 (GND)
- new net /ATTRACT: UD1.3, UD2.1
- new net /RUN: D4.2 (A), R12.1, UD2.3
- new net /SRST: D4.1 (K), D5.2 (A), SW1.3 (C), UC9.12, UC9.5
- new net /STOPG1: UB2.1
- new net /STOPG2: UB2.2
Other:
- company: (none) -> Atari
- title: (none) -> PONG

Commit message: R20260918
Parts:
- D3, D4, D5: footprint (none) -> Diode_THT:D_DO-35_SOD27_P10.16mm_Horizontal
- UB2, UC9, UD1, UD2, UE4, UE5, UE6, UG3: footprint Package_DIP:DIP-14_W7.62mm_Socket_LongPads -> pong:pong_DIP-14_W7.62mm_Socket_LongPads
- renumbered SW1 to SW2
Connections:
- net +5V is gone; now on net +3.3V: UC9.14 (VCC), UC9.14 (VCC)
- net GND: now also UE5.7 (GND), UF4.1 (GND), UF4.5 (CONT), UF4.6 (THRES), UF4.7 (DISCH)
- net /RUN: now also UE5.1
- net /SRST: now also UE6.4
- net /MISS: now reaches UE6.5
- net RST SPEED: now reaches UE6.6
- net RST SPEED: now also UE6.1, UE6.2
- net PAD1: now reaches UG3.1
- net at UG3.2: now also UG3.12
- net at UG3.3: now also UB2.9
- net at UE5.13: now also UF4.3 (OUT)
- net +3.3V: now reaches UE5.14 (VCC)
- net +3.3V: now also UD1.14 (VCC), UE4.14 (VCC)
- net STOP G: now reaches UE5.2
- net at UG3.11: now also UB2.10
- net PAD2: now reaches UG3.13
- net at UF4.2 (TRIG): now also UE6.3
- net at UF4.4 (~{RST}): now also UF4.8 (VCC)
- net HIT: now reaches UB2.8
Other:
- note added: "NEED G1B"
- moved on the sheet: D3, UE5A, UE6A, UE6B, UF4, UG3D

Commit message: R20260922
Parts:
- C10: footprint (none) -> Capacitor_THT:C_Axial_L3.8mm_D2.6mm_P10.00mm_Horizontal
- D5: value 1N914 -> 1N4001; footprint Diode_THT:D_DO-35_SOD27_P10.16mm_Horizontal -> Diode_THT:D_DO-41_SOD81_P10.16mm_Horizontal
- R12, R13, R8, R9: footprint (none) -> Resistor_THT:R_Axial_DIN0207_L6.3mm_D2.5mm_P10.16mm_Horizontal
Changed lines of the file:
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@@
 			)
 		)
-		(property "Footprint" ""
+		(property "Footprint" "Resistor_THT:R_Axial_DIN0207_L6.3mm_D2.5mm_P10.16mm_Horizontal"
 			(at 101.854 96.774 90)
 			(hide yes)
@@
 			)
 		)
-		(property "Value" "1N914"
+		(property "Value" "1N4001"
 			(at 44.45 96.5199 90)
 			(show_name no)
@@
 			)
 		)
-		(property "Footprint" "Diode_THT:D_DO-35_SOD27_P10.16mm_Horizontal"
+		(property "Footprint" "Diode_THT:D_DO-41_SOD81_P10.16mm_Horizontal"
 			(at 41.91 95.25 0)
 			(hide yes)
@@
 			)
 		)
-		(property "Footprint" ""
+		(property "Footprint" "Capacitor_THT:C_Axial_L3.8mm_D2.6mm_P10.00mm_Horizontal"
 			(at 78.74 87.3252 0)
 			(hide yes)
@@
 			)
 		)
-		(property "Footprint" ""
+		(property "Footprint" "Resistor_THT:R_Axial_DIN0207_L6.3mm_D2.5mm_P10.16mm_Horizontal"
 			(at 70.104 96.266 90)
 			(hide yes)
@@
 			)
 		)
-		(property "Footprint" ""
+		(property "Footprint" "Resistor_THT:R_Axial_DIN0207_L6.3mm_D2.5mm_P10.16mm_Horizontal"
 			(at 104.394 114.046 90)
 			(hide yes)
@@
 			)
 		)
-		(property "Footprint" ""
+		(property "Footprint" "Resistor_THT:R_Axial_DIN0207_L6.3mm_D2.5mm_P10.16mm_Horizontal"
 			(at 87.376 79.756 90)
 			(hide yes)

Commit message: R20260922PM
Parts:
- added Q1: 2N3644, symbol Transistor_BJT:Q_NPN_EBC
- added Q2, Q3: 2N3643, symbol Transistor_BJT:Q_NPN_EBC
- C10: value C -> .1
Connections:
- net GND: now also Q1.3 (C)
- net at R8.1: now also Q1.1 (E)
- net at C10.2, R12.2, R13.2: now also Q1.2 (B)

Commit message: R20260924
Parts:
- added C22, C24: .1, Capacitor_THT:C_Axial_L3.8mm_D2.6mm_P10.00mm_Horizontal, symbol Device:C
- added C23: 4.7, Capacitor_THT:C_Axial_L3.8mm_D2.6mm_P10.00mm_Horizontal, symbol Device:C_Polarized_US
- added D8: 1N914, Diode_THT:D_DO-35_SOD27_P10.16mm_Horizontal, symbol Device:D
- added R32: 100, Resistor_THT:R_Axial_DIN0207_L6.3mm_D2.5mm_P10.16mm_Horizontal, symbol Device:R_US
- added R33: 330k, Resistor_THT:R_Axial_DIN0207_L6.3mm_D2.5mm_P10.16mm_Horizontal, symbol Device:R_US
Connections:
- net GND: now also Q2.3 (C), Q3.3 (C), C22.2, C23.2, C24.2, D8.2 (A), R32.1; no longer UF4.5 (CONT), UF4.6 (THRES), UF4.7 (DISCH)
- net /RUN: now also Q2.1 (E)
- net at Q3.1 (E): now also Q2.2 (B), R9.1, C22.1, R32.2
- net 15: now reaches Q3.2 (B)
- net 15: now also D8.1 (K)
- net 12: now reaches SW2.1 (A), UC9.13, UC9.6
- net +5V: now reaches UF4.4 (~{RST}), UF4.8 (VCC)
- net +5V: now also R33.2
- net /SRST renamed 10
- new net: C23.1, C24.1, R33.1, UF4.5 (CONT), UF4.6 (THRES), UF4.7 (DISCH)
Other:
- moved on the sheet: Q2, Q3, R9, UC9C
