File: PADDLE1.kicad_sch (KiCad schematic)
At the start: 10 parts

Commit message: Added remainder of sheets
Parts:
- UB7, UB8, UC9: footprint Package_DIP:DIP-14_W10.16mm -> Package_DIP:DIP-14_W7.62mm_Socket_LongPads
- UB9: footprint Package_DIP:DIP-8_W7.62mm -> Package_DIP:DIP-8_W7.62mm_Socket_LongPads
Changed lines of the file:
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@@
 			)
 		)
-		(property "Footprint" "Package_DIP:DIP-14_W10.16mm"
+		(property "Footprint" "Package_DIP:DIP-14_W7.62mm_Socket_LongPads"
 			(at 125.73 66.04 0)
 			(hide yes)
@@
 			)
 		)
-		(property "Footprint" "Package_DIP:DIP-14_W10.16mm"
+		(property "Footprint" "Package_DIP:DIP-14_W7.62mm_Socket_LongPads"
 			(at 156.21 87.63 0)
 			(hide yes)
@@
 			)
 		)
-		(property "Footprint" "Package_DIP:DIP-8_W7.62mm"
+		(property "Footprint" "Package_DIP:DIP-8_W7.62mm_Socket_LongPads"
 			(at 85.09 90.17 0)
 			(hide yes)
@@
 			)
 		)
-		(property "Footprint" "Package_DIP:DIP-14_W10.16mm"
+		(property "Footprint" "Package_DIP:DIP-14_W7.62mm_Socket_LongPads"
 			(at 156.21 68.58 0)
 			(hide yes)
@@
 			)
 		)
-		(property "Footprint" "Package_DIP:DIP-14_W10.16mm"
+		(property "Footprint" "Package_DIP:DIP-14_W7.62mm_Socket_LongPads"
 			(at 109.22 111.76 0)
 			(hide yes)

Commit message: R20260915
Parts:
- R10: value 56K -> R_US; symbol Device:R -> Device:R_US
- R11: value 470 -> R_US; symbol Device:R -> Device:R_US
- UA7: footprint (none) -> Package_DIP:DIP-14_W7.62mm_Socket_LongPads
Connections:
- net GND: now also UA7.7 (GND), UB8.10 (GND), UB9.1 (GND)
- net +3.3V: now reaches UA7.14 (VCC)
- net +3.3V: now also UB8.5 (VCC), UC9.14 (VCC)
Other:
- company: (none) -> Atari
- title: (none) -> PONG
- moved on the sheet: C8, UA7B, UB8

Commit message: R20260918
Parts:
- R10: value R_US -> 56K
- UA7, UB7, UB8, UC9: footprint Package_DIP:DIP-14_W7.62mm_Socket_LongPads -> pong:pong_DIP-14_W7.62mm_Socket_LongPads
Connections:
- net at UA7.10, UB8.12 (Q0): now also UB8.1 (~{CKB})
- net at C8.2, R10.2, UB9.6 (THRES): now also UB9.7 (DISCH)
Other:
- moved on the sheet: C8
Changed lines of the file:
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@@
+	)
+	(junction
+		(at 109.22 144.78)
+		(diameter 0)
+		(color 0 0 0 0)
+	)
+	(junction
+		(at 49.53 68.58)
+		(diameter 0)
+		(color 0 0 0 0)
 	)
 	(junction
@@
 	)
 	(junction
-		(at 49.53 68.58)
+		(at 49.53 77.47)
 		(diameter 0)
 		(color 0 0 0 0)
@@
 	(wire
 		(pts
+			(xy 99.06 95.25) (xy 74.93 95.25)
+		)
+		(stroke
+			(width 0)
+			(type default)
+		)
+	)
+	(wire
+		(pts
 			(xy 109.22 92.71) (xy 109.22 95.25)
 		)
@@
 	(wire
 		(pts
+			(xy 74.93 63.5) (xy 59.69 63.5)
+		)
+		(stroke
+			(width 0)
+			(type default)
+		)
+	)
+	(wire
+		(pts
 			(xy 87.63 52.07) (xy 64.77 52.07)
 		)
@@
 	(wire
 		(pts
+			(xy 74.93 144.78) (xy 109.22 144.78)
+		)
+		(stroke
+			(width 0)
+			(type default)
+		)
+	)
+	(wire
+		(pts
+			(xy 74.93 95.25) (xy 74.93 144.78)
+		)
+		(stroke
+			(width 0)
+			(type default)
+		)
+	)
+	(wire
+		(pts
 			(xy 109.22 135.89) (xy 109.22 144.78)
 		)
@@
 	(wire
 		(pts
+			(xy 49.53 77.47) (xy 49.53 68.58)
+		)
+		(stroke
+			(width 0)
+			(type default)
+		)
+	)
+	(wire
+		(pts
 			(xy 49.53 49.53) (xy 49.53 54.61)
 		)
@@
 	(wire
 		(pts
+			(xy 59.69 63.5) (xy 59.69 77.47)
+		)
+		(stroke
+			(width 0)
+			(type default)
+		)
+	)
+	(wire
+		(pts
 			(xy 64.77 60.96) (xy 64.77 52.07)
 		)
@@
 	(wire
 		(pts
+			(xy 59.69 77.47) (xy 49.53 77.47)
+		)
+		(stroke
+			(width 0)
+			(type default)
+		)
+	)
+	(wire
+		(pts
 			(xy 74.93 60.96) (xy 64.77 60.96)
 		)
@@
 	(wire
 		(pts
-			(xy 49.53 73.66) (xy 49.53 68.58)
-		)
-		(stroke
-			(width 0)
-			(type default)
-		)
-	)
-	(wire
-		(pts
-			(xy 63.5 71.12) (xy 74.93 71.12)
+			(xy 49.53 82.55) (xy 49.53 77.47)
 		)
 		(stroke
@@
 	(global_label "{slash}256V"
 		(shape input)
-		(at 63.5 71.12 180)
+		(at 74.93 71.12 180)
 		(fields_autoplaced yes)
 		(effects
@@
 		)
 		(property "Intersheetrefs" "${INTERSHEET_REFS}"
-			(at 54.4672 71.12 0)
+			(at 65.8972 71.12 0)
 			(hide yes)
 			(show_name no)
@@
 			)
 		)
-		(property "Footprint" "Package_DIP:DIP-14_W7.62mm_Socket_LongPads"
+		(property "Footprint" "pong:pong_DIP-14_W7.62mm_Socket_LongPads"
 			(at 167.64 147.32 0)
 			(hide yes)
@@
 			)
 		)
-		(property "Footprint" "Package_DIP:DIP-14_W7.62mm_Socket_LongPads"
+		(property "Footprint" "pong:pong_DIP-14_W7.62mm_Socket_LongPads"
 			(at 125.73 66.04 0)
 			(hide yes)
@@
 			)
 		)
-		(property "Footprint" "Package_DIP:DIP-14_W7.62mm_Socket_LongPads"
+		(property "Footprint" "pong:pong_DIP-14_W7.62mm_Socket_LongPads"
 			(at 156.21 87.63 0)
 			(hide yes)
@@
 			)
 		)
-		(property "Footprint" "Package_DIP:DIP-14_W7.62mm_Socket_LongPads"
+		(property "Footprint" "pong:pong_DIP-14_W7.62mm_Socket_LongPads"
 			(at 156.21 68.58 0)
 			(hide yes)
@@
 			)
 		)
-		(property "Footprint" "Package_DIP:DIP-14_W7.62mm_Socket_LongPads"
+		(property "Footprint" "pong:pong_DIP-14_W7.62mm_Socket_LongPads"
 			(at 109.22 115.57 0)
 			(hide yes)
@@
 	(symbol
 		(lib_id "Device:C")
-		(at 49.53 77.47 180)
+		(at 49.53 86.36 180)
 		(unit 1)
 		(body_style 1)
@@
 		(fields_autoplaced yes)
 		(property "Reference" "C8"
-			(at 53.34 76.1999 0)
+			(at 53.34 85.0899 0)
 			(show_name no)
 			(do_not_autoplace no)
@@
 		)
 		(property "Value" ".1uF"
-			(at 53.34 78.7399 0)
+			(at 53.34 87.6299 0)
 			(show_name no)
 			(do_not_autoplace no)
@@
 		)
 		(property "Footprint" ""
-			(at 48.5648 73.66 0)
+			(at 48.5648 82.55 0)
 			(hide yes)
 			(show_name no)
@@
 		)
 		(property "Datasheet" ""
-			(at 49.53 77.47 0)
+			(at 49.53 86.36 0)
 			(hide yes)
 			(show_name no)
@@
 		)
 		(property "Description" "Unpolarized capacitor"
-			(at 49.53 77.47 0)
+			(at 49.53 86.36 0)
 			(hide yes)
 			(show_name no)
@@
 			)
 		)
-		(property "Value" "R_US"
+		(property "Value" "56K"
 			(at 52.07 59.6899 0)
 			(show_name no)
@@
 	(symbol
 		(lib_id "power:GND")
-		(at 49.53 81.28 0)
+		(at 49.53 90.17 0)
 		(unit 1)
 		(body_style 1)
@@
 		(fields_autoplaced yes)
 		(property "Reference" "#PWR014"
-			(at 49.53 87.63 0)
+			(at 49.53 96.52 0)
 			(hide yes)
 			(show_name no)
@@
 		)
 		(property "Value" "GND"
-			(at 49.53 86.36 0)
+			(at 49.53 95.25 0)
 			(show_name no)
 			(do_not_autoplace no)
@@
 		)
 		(property "Footprint" ""
-			(at 49.53 81.28 0)
+			(at 49.53 90.17 0)
 			(hide yes)
 			(show_name no)
@@
 		)
 		(property "Datasheet" ""
-			(at 49.53 81.28 0)
+			(at 49.53 90.17 0)
 			(hide yes)
 			(show_name no)
@@
 		)
 		(property "Description" "Power symbol creates a global label with name \"GND\" , ground"
-			(at 49.53 81.28 0)
-			(hide yes)
-			(show_name no)
+			(at 49.53 90.17 0)
+			(hide yes)
+			(show_name no)

Commit message: R20260922
Parts:
- added D7: 1N914, Diode_THT:D_DO-35_SOD27_P10.16mm_Horizontal, symbol Diode:1N914
- C8: footprint (none) -> Capacitor_THT:C_Axial_L3.8mm_D2.6mm_P12.50mm_Horizontal
- C9: footprint (none) -> Capacitor_THT:C_Axial_L3.8mm_D2.6mm_P10.00mm_Horizontal
- R10: footprint (none) -> Resistor_THT:R_Axial_DIN0207_L6.3mm_D2.5mm_P10.16mm_Horizontal
- R11: value R_US -> R; footprint (none) -> Resistor_THT:R_Axial_DIN0207_L6.3mm_D2.5mm_P10.16mm_Horizontal
Connections:
- net at C8.2, R10.2, UB9.6 (THRES): now also D7.2 (A); no longer UB9.7 (DISCH)
- new net: D7.1 (K), UB9.7 (DISCH)
Changed lines of the file:
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@@
+	(wire
+		(pts
+			(xy 50.8 77.47) (xy 49.53 77.47)
+		)
+		(stroke
+			(width 0)
+			(type default)
+		)
+	)
 	(wire
 		(pts
@@
 	(wire
 		(pts
-			(xy 59.69 77.47) (xy 49.53 77.47)
+			(xy 59.69 77.47) (xy 58.42 77.47)
 		)
 		(stroke
@@
 			)
 		)
-		(property "Footprint" ""
+		(property "Footprint" "Capacitor_THT:C_Axial_L3.8mm_D2.6mm_P10.00mm_Horizontal"
 			(at 100.6348 24.13 0)
 			(hide yes)
@@
 	)
 	(symbol
+		(lib_id "Diode:1N914")
+		(at 54.61 77.47 180)
+		(unit 1)
+		(body_style 1)
+		(exclude_from_sim no)
+		(in_bom yes)
+		(on_board yes)
+		(in_pos_files yes)
+		(dnp no)
+		(fields_autoplaced yes)
+		(property "Reference" "D7"
+			(at 54.61 71.12 0)
+			(show_name no)
+			(do_not_autoplace no)
+			(effects
+				(font
+					(size 1.27 1.27)
+				)
+			)
+		)
+		(property "Value" "1N914"
+			(at 54.61 73.66 0)
+			(show_name no)
+			(do_not_autoplace no)
+			(effects
+				(font
+					(size 1.27 1.27)
+				)
+			)
+		)
+		(property "Footprint" "Diode_THT:D_DO-35_SOD27_P10.16mm_Horizontal"
+			(at 54.61 73.025 0)
+			(hide yes)
+			(show_name no)
+			(do_not_autoplace no)
+			(effects
+				(font
+					(size 1.27 1.27)
+				)
+			)
+		)
+		(property "Datasheet" "http://www.vishay.com/docs/85622/1n914.pdf"
+			(at 54.61 77.47 0)
+			(hide yes)
+			(show_name no)
+			(do_not_autoplace no)
+			(effects
+				(font
+					(size 1.27 1.27)
+				)
+			)
+		)
+		(property "Description" "100V 0.3A Small Signal Fast Switching Diode, DO-35"
+			(at 54.61 77.47 0)
+			(hide yes)
+			(show_name no)
+			(do_not_autoplace no)
+			(effects
+				(font
+					(size 1.27 1.27)
+				)
+			)
+		)
+		(property "Sim.Device" "D"
+			(at 54.61 77.47 0)
+			(hide yes)
+			(show_name no)
+			(do_not_autoplace no)
+			(effects
+				(font
+					(size 1.27 1.27)
+				)
+			)
+		)
+		(property "Sim.Pins" "1=K 2=A"
+			(at 54.61 77.47 0)
+			(hide yes)
+			(show_name no)
+			(do_not_autoplace no)
+			(effects
+				(font
+					(size 1.27 1.27)
+				)
+			)
+		)
+		(pin "2"
+		)
+		(pin "1"
+		)
+		(instances
+			(project "pong"
+				(path "/6c55baa6-be38-444e-ac95-9cecf812b759/f8442d93-e578-41b1-a001-24e7a8b1cfac"
+					(reference "D7")
+					(unit 1)
+				)
+			)
+		)
+	)
+	(symbol
 		(lib_id "Device:C")
 		(at 49.53 86.36 180)
@@
 			)
 		)
-		(property "Footprint" ""
+		(property "Footprint" "Capacitor_THT:C_Axial_L3.8mm_D2.6mm_P12.50mm_Horizontal"
 			(at 48.5648 82.55 0)
 			(hide yes)
@@
 			)
 		)
-		(property "Value" "R_US"
+		(property "Value" "R"
 			(at 87.63 44.4499 0)
 			(show_name no)
@@
 			)
 		)
-		(property "Footprint" ""
+		(property "Footprint" "Resistor_THT:R_Axial_DIN0207_L6.3mm_D2.5mm_P10.16mm_Horizontal"
 			(at 86.106 43.434 90)
 			(hide yes)
@@
 			)
 		)
-		(property "Footprint" ""
+		(property "Footprint" "Resistor_THT:R_Axial_DIN0207_L6.3mm_D2.5mm_P10.16mm_Horizontal"
 			(at 50.546 58.674 90)
 			(hide yes)

Commit message: R20260924
Connections:
- net 19: now reaches C9.2, R11.1
Changed lines of the file:
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@@
+	)
+	(junction
+		(at 85.09 24.13)
+		(diameter 0)
+		(color 0 0 0 0)
 	)
 	(junction
@@
 		(pts
 			(xy 74.93 95.25) (xy 74.93 144.78)
+		)
+		(stroke
+			(width 0)
+			(type default)
+		)
+	)
+	(wire
+		(pts
+			(xy 64.77 24.13) (xy 85.09 24.13)
 		)
 		(stroke
@@
 			(hide yes)
 			(show_name no)
+			(do_not_autoplace no)
+			(effects
+				(font
+					(size 1.27 1.27)
+				)
+				(justify left)
+			)
+		)
+	)
+	(global_label "19"
+		(shape input)
+		(at 71.12 24.13 90)
+		(fields_autoplaced yes)
+		(effects
+			(font
+				(size 1.27 1.27)
+			)
+			(justify left)
+		)
+		(property "Intersheetrefs" "${INTERSHEET_REFS}"
+			(at 71.12 18.7258 90)
+			(hide yes)
+			(show_name no)
